File: Projects/CANBoard/CANBus.sch (KiCad schematic (older format))
At the start: 11 parts, among them J1_CAN1 HEADER_4, J2_CAN1 HEADER_4, J3_CAN1 HEADER_4, J4_CAN1 HEADER_4, J5_CAN1 HEADER_4, J6_CAN1 HEADER_4, U1_CAN1 MCP2562, U2_CAN1 MCP2515

Commit message: Major updates for power distribution and Communications boards
Parts:
- C1_CAN1, C2_CAN1: footprint (none) -> Capacitors_ThroughHole:C_Radial_D5_L11_P2.5
- J1_CAN1, J2_CAN1, J3_CAN1, J4_CAN1, J5_CAN1, J6_CAN1: footprint (none) -> Pin_Headers:Pin_Header_Straight_1x04
- R1_CAN1: footprint (none) -> Resistors_ThroughHole:Resistor_Horizontal_RM10mm
- U1_CAN1: footprint (none) -> Housings_DIP:DIP-8_W7.62mm
- U2_CAN1: footprint (none) -> Housings_DIP:DIP-18_W7.62mm
Changed lines of the file:
@@
 LIBS:valves
 LIBS:USSTComponents
-LIBS:w_analog
-LIBS:w_connectors
-LIBS:w_device
-LIBS:w_logic
-LIBS:w_memory
-LIBS:w_microcontrollers
-LIBS:w_opto
-LIBS:w_relay
-LIBS:w_rtx
-LIBS:w_transistor
-LIBS:w_vacuum
 LIBS:PiMainboard-cache
 EELAYER 25 0
@@
 $Descr A4 11693 8268
 encoding utf-8
-Sheet 9 10
+Sheet 2 3
 Title ""
 Date ""
@@
 AR Path="/567C9351/568AC62D" Ref="U2_CAN1"  Part="1"
 AR Path="/56EDDFF0/56EF4FC7/568AC62D" Ref="U2_CAN1"  Part="1"
+AR Path="/56EF4FC7/568AC62D" Ref="U2_CAN1"  Part="1"
 F 0 "U2_CAN1" H 6650 5300 60  0000 C CNN
 F 1 "MCP2515" H 6400 4200 60  0000 C CNN
-F 2 "" H 6350 4650 60  0000 C CNN
+F 2 "Housings_DIP:DIP-18_W7.62mm" H 6350 4650 60  0001 C CNN
 F 3 "" H 6350 4650 60  0000 C CNN
 	1    6450 4750
@@
 AR Path="/567C9351/568AC6C6" Ref="U1_CAN1"  Part="1"
 AR Path="/56EDDFF0/56EF4FC7/568AC6C6" Ref="U1_CAN1"  Part="1"
+AR Path="/56EF4FC7/568AC6C6" Ref="U1_CAN1"  Part="1"
 F 0 "U1_CAN1" H 6600 4050 60  0000 C CNN
 F 1 "MCP2562" H 6400 3450 60  0000 C CNN
-F 2 "" H 6150 3650 60  0000 C CNN
+F 2 "Housings_DIP:DIP-8_W7.62mm" H 6150 3650 60  0001 C CNN
 F 3 "" H 6150 3650 60  0000 C CNN
 	1    6400 3750
@@
 AR Path="/567C9351/568ACA60" Ref="C1_CAN1"  Part="1"
 AR Path="/56EDDFF0/56EF4FC7/568ACA60" Ref="C1_CAN1"  Part="1"
+AR Path="/56EF4FC7/568ACA60" Ref="C1_CAN1"  Part="1"
 F 0 "C1_CAN1" H 7700 4510 50  0000 L CNN
 F 1 "0.1uF" H 7700 4440 50  0000 L CNN
-F 2 "" H 7650 4500 60  0000 C CNN
+F 2 "Capacitors_ThroughHole:C_Radial_D5_L11_P2.5" H 7650 4500 60  0001 C CNN
 F 3 "" H 7650 4500 60  0000 C CNN
 	1    7650 4500
@@
 AR Path="/567C9351/568ACCF6" Ref="C2_CAN1"  Part="1"
 AR Path="/56EDDFF0/56EF4FC7/568ACCF6" Ref="C2_CAN1"  Part="1"
+AR Path="/56EF4FC7/568ACCF6" Ref="C2_CAN1"  Part="1"
 F 0 "C2_CAN1" H 5250 3760 50  0000 L CNN
 F 1 "0.1uF" H 5250 3690 50  0000 L CNN
-F 2 "" H 5200 3750 60  0000 C CNN
+F 2 "Capacitors_ThroughHole:C_Radial_D5_L11_P2.5" H 5200 3750 60  0001 C CNN
 F 3 "" H 5200 3750 60  0000 C CNN
 	1    5200 3750
@@
 AR Path="/567C9351/568AD3DE" Ref="J1_CAN1"  Part="1"
 AR Path="/56EDDFF0/56EF4FC7/568AD3DE" Ref="J1_CAN1"  Part="1"
+AR Path="/56EF4FC7/568AD3DE" Ref="J1_CAN1"  Part="1"
 F 0 "J1_CAN1" H 9850 2400 60  0000 C CNN
 F 1 "HEADER_4" H 9850 1900 60  0000 C CNN
-F 2 "" H 9850 2150 60  0000 C CNN
+F 2 "Pin_Headers:Pin_Header_Straight_1x04" H 9850 2150 60  0001 C CNN
 F 3 "" H 9850 2150 60  0000 C CNN
 	1    9850 2150
@@
 AR Path="/567C9351/568ADD75" Ref="J2_CAN1"  Part="1"
 AR Path="/56EDDFF0/56EF4FC7/568ADD75" Ref="J2_CAN1"  Part="1"
+AR Path="/56EF4FC7/568ADD75" Ref="J2_CAN1"  Part="1"
 F 0 "J2_CAN1" H 9850 3050 60  0000 C CNN
 F 1 "HEADER_4" H 9850 2550 60  0000 C CNN
-F 2 "" H 9850 2800 60  0000 C CNN
+F 2 "Pin_Headers:Pin_Header_Straight_1x04" H 9850 2800 60  0001 C CNN
 F 3 "" H 9850 2800 60  0000 C CNN
 	1    9850 2800
@@
 AR Path="/567C9351/568ADF7B" Ref="J3_CAN1"  Part="1"
 AR Path="/56EDDFF0/56EF4FC7/568ADF7B" Ref="J3_CAN1"  Part="1"
+AR Path="/56EF4FC7/568ADF7B" Ref="J3_CAN1"  Part="1"
 F 0 "J3_CAN1" H 9850 3700 60  0000 C CNN
 F 1 "HEADER_4" H 9850 3200 60  0000 C CNN
-F 2 "" H 9850 3450 60  0000 C CNN
+F 2 "Pin_Headers:Pin_Header_Straight_1x04" H 9850 3450 60  0001 C CNN
 F 3 "" H 9850 3450 60  0000 C CNN
 	1    9850 3450
@@
 AR Path="/567C9351/568ADF89" Ref="J4_CAN1"  Part="1"
 AR Path="/56EDDFF0/56EF4FC7/568ADF89" Ref="J4_CAN1"  Part="1"
+AR Path="/56EF4FC7/568ADF89" Ref="J4_CAN1"  Part="1"
 F 0 "J4_CAN1" H 9850 4350 60  0000 C CNN
 F 1 "HEADER_4" H 9850 3850 60  0000 C CNN
-F 2 "" H 9850 4100 60  0000 C CNN
+F 2 "Pin_Headers:Pin_Header_Straight_1x04" H 9850 4100 60  0001 C CNN
 F 3 "" H 9850 4100 60  0000 C CNN
 	1    9850 4100
@@
 AR Path="/567C9351/568AE0B5" Ref="J5_CAN1"  Part="1"
 AR Path="/56EDDFF0/56EF4FC7/568AE0B5" Ref="J5_CAN1"  Part="1"
+AR Path="/56EF4FC7/568AE0B5" Ref="J5_CAN1"  Part="1"
 F 0 "J5_CAN1" H 9850 5000 60  0000 C CNN
 F 1 "HEADER_4" H 9850 4500 60  0000 C CNN
-F 2 "" H 9850 4750 60  0000 C CNN
+F 2 "Pin_Headers:Pin_Header_Straight_1x04" H 9850 4750 60  0001 C CNN
 F 3 "" H 9850 4750 60  0000 C CNN
 	1    9850 4750
@@
 AR Path="/567C9351/568AE0C3" Ref="J6_CAN1"  Part="1"
 AR Path="/56EDDFF0/56EF4FC7/568AE0C3" Ref="J6_CAN1"  Part="1"
+AR Path="/56EF4FC7/568AE0C3" Ref="J6_CAN1"  Part="1"
 F 0 "J6_CAN1" H 9850 5650 60  0000 C CNN
 F 1 "HEADER_4" H 9850 5150 60  0000 C CNN
-F 2 "" H 9850 5400 60  0000 C CNN
+F 2 "Pin_Headers:Pin_Header_Straight_1x04" H 9850 5400 60  0001 C CNN
 F 3 "" H 9850 5400 60  0000 C CNN
 	1    9850 5400
@@
 AR Path="/56EDDFF0/56EF4FC7/56EF1C19" Ref="R1_CAN1"  Part="1"
 AR Path="/567C9351/56EF1C19" Ref="R1_CAN1"  Part="1"
+AR Path="/56EF4FC7/56EF1C19" Ref="R1_CAN1"  Part="1"
 F 0 "R1_CAN1" V 7430 2600 50  0000 C CNN
 F 1 "100" V 7350 2600 50  0000 C CNN
-F 2 "" V 7280 2600 50  0000 C CNN
+F 2 "Resistors_ThroughHole:Resistor_Horizontal_RM10mm" V 7280 2600 50  0001 C CNN
 F 3 "" H 7350 2600 50  0000 C CNN
 	1    7350 2600
@@
 	7150 3900 7150 4350
 Wire Wire Line
-	7000 4350 7150 4350
-Wire Wire Line
-	7150 4350 7650 4350
-Wire Wire Line
-	7650 4350 7900 4350
+	7000 4350 7900 4350
 Connection ~ 7150 4350
 Wire Wire Line
@@
 	5500 3700 5500 3600
 Wire Wire Line
-	5500 3600 5200 3600
-Wire Wire Line
-	5200 3600 5050 3600
+	5500 3600 5050 3600
 Wire Wire Line
 	5200 3600 5200 3700
@@
 	5500 3800 5500 3900
 Wire Wire Line
-	5500 3900 5200 3900
-Wire Wire Line
-	5200 3900 5050 3900
+	5500 3900 5050 3900
 Wire Wire Line
 	5200 3900 5200 3850
