File: Projects/VESC/design/BLDC_4.sch (KiCad schematic (older format))
At the start: 26 parts, among them K1 SERVO, P1 HALL/Encoder, P101 CANBUS, P3 PWR_COMM, P4 IN+, P5 IN-, P6 MOTOR1, P7 MOTOR2, P9 MOTOR3, X1 MINI-USB-SHIELD-32005-201

Commit message: Started making changes to VESC layout and schematic
Parts:
- C2, C3: footprint CRF1:SMD-0603_c -> Capacitors_SMD:C_0805
- D1, D2, D3: footprint LEDs:LED-0603 -> LEDs:LED_0805
- R103, R104, R22, R3, R37, R38, R4, R5, R6: footprint CRF1:SMD-0603_r -> Resistors_SMD:R_0805
Changed lines of the file:
@@
 $EndComp
 $Comp
-L +5V #PWR01
+L +5V #PWR3
 U 1 1 522DA04D
 P 1450 4900
-F 0 "#PWR01" H 1450 4990 20  0001 C CNN
+F 0 "#PWR3" H 1450 4990 20  0001 C CNN
 F 1 "+5V" V 1400 4950 30  0000 C CNN
 F 2 "" H 1450 4900 60  0001 C CNN
@@
 $EndComp
 $Comp
-L GND-RESCUE-BLDC_4 #PWR02
+L GND-RESCUE-BLDC_4 #PWR5
 U 1 1 522DA053
 P 1500 4400
-F 0 "#PWR02" H 1500 4400 30  0001 C CNN
+F 0 "#PWR5" H 1500 4400 30  0001 C CNN
 F 1 "GND" H 1500 4330 30  0001 C CNN
 F 2 "" H 1500 4400 60  0001 C CNN
@@
 F 0 "C3" V 6600 5850 50  0000 L CNN
 F 1 "100n" V 6600 5500 50  0000 L CNN
-F 2 "CRF1:SMD-0603_c" H 6550 5750 60  0001 C CNN
+F 2 "Capacitors_SMD:C_0805" H 6550 5750 60  0001 C CNN
 F 3 "" H 6550 5750 60  0001 C CNN
 	1    6550 5750
@@
 F 0 "R5" V 6500 5500 50  0000 C CNN
 F 1 "2k2" V 6600 5550 50  0000 C CNN
-F 2 "CRF1:SMD-0603_r" H 6600 5550 60  0001 C CNN
+F 2 "Resistors_SMD:R_0805" H 6600 5550 60  0001 C CNN
 F 3 "" H 6600 5550 60  0001 C CNN
 	1    6600 5550
@@
 F 0 "C2" V 2100 2500 50  0000 L CNN
 F 1 "100n" V 2100 2150 50  0000 L CNN
-F 2 "CRF1:SMD-0603_c" H 2050 2400 60  0001 C CNN
+F 2 "Capacitors_SMD:C_0805" H 2050 2400 60  0001 C CNN
 F 3 "" H 2050 2400 60  0001 C CNN
 	1    2050 2400
@@
 $EndComp
 $Comp
-L GND-RESCUE-BLDC_4 #PWR03
+L GND-RESCUE-BLDC_4 #PWR16
 U 1 1 522DA0BA
 P 7000 5850
-F 0 "#PWR03" H 7000 5850 30  0001 C CNN
+F 0 "#PWR16" H 7000 5850 30  0001 C CNN
 F 1 "GND" H 7000 5780 30  0001 C CNN
 F 2 "" H 7000 5850 60  0001 C CNN
@@
 V_SUPPLY
 $Comp
-L GND-RESCUE-BLDC_4 #PWR04
+L GND-RESCUE-BLDC_4 #PWR9
 U 1 1 522DA0CE
 P 1700 2500
-F 0 "#PWR04" H 1700 2500 30  0001 C CNN
+F 0 "#PWR9" H 1700 2500 30  0001 C CNN
 F 1 "GND" H 1700 2430 30  0001 C CNN
 F 2 "" H 1700 2500 60  0001 C CNN
@@
 F 0 "R4" V 2000 2050 50  0000 C CNN
 F 1 "2k2" V 2050 2250 50  0000 C CNN
-F 2 "CRF1:SMD-0603_r" H 2050 2250 60  0001 C CNN
+F 2 "Resistors_SMD:R_0805" H 2050 2250 60  0001 C CNN
 F 3 "" H 2050 2250 60  0001 C CNN
 	1    2050 2250
@@
 F 0 "R3" V 2000 1950 50  0000 C CNN
 F 1 "39k" V 2050 2150 50  0000 C CNN
-F 2 "CRF1:SMD-0603_r" H 2050 2150 60  0001 C CNN
+F 2 "Resistors_SMD:R_0805" H 2050 2150 60  0001 C CNN
 F 3 "" H 2050 2150 60  0001 C CNN
 	1    2050 2150
@@
 $EndComp
 $Comp
-L GND-RESCUE-BLDC_4 #PWR05
+L GND-RESCUE-BLDC_4 #PWR4
 U 1 1 522DA0E2
 P 1450 5450
-F 0 "#PWR05" H 1450 5450 30  0001 C CNN
+F 0 "#PWR4" H 1450 5450 30  0001 C CNN
 F 1 "GND" H 1450 5380 30  0001 C CNN
 F 2 "" H 1450 5450 60  0001 C CNN
@@
 $EndComp
 $Comp
-L GND-RESCUE-BLDC_4 #PWR06
+L GND-RESCUE-BLDC_4 #PWR8
 U 1 1 522DA0FC
 P 1600 3450
-F 0 "#PWR06" H 1600 3450 30  0001 C CNN
+F 0 "#PWR8" H 1600 3450 30  0001 C CNN
 F 1 "GND" H 1600 3380 30  0001 C CNN
 F 2 "" H 1600 3450 60  0001 C CNN
@@
 NoConn ~ 1450 3250
 $Comp
-L +5V #PWR07
+L +5V #PWR6
 U 1 1 522DA11A
 P 1550 5250
-F 0 "#PWR07" H 1550 5340 20  0001 C CNN
+F 0 "#PWR6" H 1550 5340 20  0001 C CNN
 F 1 "+5V" V 1550 5400 30  0000 C CNN
 F 2 "" H 1550 5250 60  0001 C CNN
@@
 $EndComp
 $Comp
-L VCC #PWR08
+L VCC #PWR7
 U 1 1 522DA120
 P 1550 5350
-F 0 "#PWR08" H 1550 5450 30  0001 C CNN
+F 0 "#PWR7" H 1550 5450 30  0001 C CNN
 F 1 "VCC" V 1550 5500 30  0000 C CNN
 F 2 "" H 1550 5350 60  0001 C CNN
@@
 $EndComp
 $Comp
-L +5V #PWR09
+L +5V #PWR15
 U 1 1 522DA158
 P 7000 5400
-F 0 "#PWR09" H 7000 5490 20  0001 C CNN
+F 0 "#PWR15" H 7000 5490 20  0001 C CNN
 F 1 "+5V" H 7000 5490 30  0000 C CNN
 F 2 "" H 7000 5400 60  0001 C CNN
@@
 F 0 "R6" V 2350 2750 50  0000 C CNN
 F 1 "0R" V 2400 2950 50  0000 C CNN
-F 2 "CRF1:SMD-0603_r" H 2400 2950 60  0001 C CNN
+F 2 "Resistors_SMD:R_0805" H 2400 2950 60  0001 C CNN
 F 3 "" H 2400 2950 60  0001 C CNN
 	1    2400 2950
@@
 $EndComp
 $Comp
-L +5V #PWR010
+L +5V #PWR10
 U 1 1 522DA254
 P 2800 2900
-F 0 "#PWR010" H 2800 2990 20  0001 C CNN
+F 0 "#PWR10" H 2800 2990 20  0001 C CNN
 F 1 "+5V" H 2800 2990 30  0000 C CNN
 F 2 "" H 2800 2900 60  0001 C CNN
@@
 $EndComp
 $Comp
-L GND-RESCUE-BLDC_4 #PWR011
+L GND-RESCUE-BLDC_4 #PWR21
 U 1 1 53FA1F8F
 P 9550 5050
-F 0 "#PWR011" H 9550 5050 30  0001 C CNN
+F 0 "#PWR21" H 9550 5050 30  0001 C CNN
 F 1 "GND" H 9550 4980 30  0001 C CNN
 F 2 "" H 9550 5050 60  0001 C CNN
@@
 $Bitmap
 Pos 10700 3200
-Scale 1,000000
+Scale 1.000000
 Data
 89 50 4E 47 0D 0A 1A 0A 00 00 00 0D 49 48 44 52 00 00 00 B9 00 00 00 C6 08 02 00 00 00 01 BB B6
@@
 C8 C8 08 D2 A9 87 39 1B F9 3D 64 10 3C A5 22 3B 19 76 2F 98 2B 2B 2B 1E 8F A7 AB AB 0B FB AC 1D
 B9 73 C8 EF 2C EC 8D 33 57 03 96 70 05 29 43 0C 6A C5 A8 D7 30 9E 87 2D DE BE E8 EA 73 2F 9C 18
-F1 B3 C3 9F 6D FA 1E FF 03 71 17 46 7E 55 DF FF 4E 00 00 00 00 49 45 4E 44 AE 42 60 82 00
+F1 B3 C3 9F 6D FA 1E FF 03 71 17 46 7E 55 DF FF 4E 00 00 00 00 49 45 4E 44 AE 42 60 82
 EndData
 $EndBitmap
@@
 $EndSheet
 $Comp
-L GND-RESCUE-BLDC_4 #PWR012
+L GND-RESCUE-BLDC_4 #PWR2
 U 1 1 53FB6DA8
 P 1450 4050
-F 0 "#PWR012" H 1450 4050 30  0001 C CNN
+F 0 "#PWR2" H 1450 4050 30  0001 C CNN
 F 1 "GND" H 1450 3980 30  0001 C CNN
 F 2 "" H 1450 4050 60  0001 C CNN
@@
 F 0 "R103" V 2350 3250 40  0000 C CNN
 F 1 "22R" V 2407 3051 40  0000 C CNN
-F 2 "CRF1:SMD-0603_r" V 2330 3050 30  0001 C CNN
+F 2 "Resistors_SMD:R_0805" V 2330 3050 30  0001 C CNN
 F 3 "" H 2400 3050 30  0000 C CNN
 	1    2400 3050
@@
 F 0 "R104" V 2350 3350 40  0000 C CNN
 F 1 "22R" V 2407 3151 40  0000 C CNN
-F 2 "CRF1:SMD-0603_r" V 2330 3150 30  0001 C CNN
+F 2 "Resistors_SMD:R_0805" V 2330 3150 30  0001 C CNN
 F 3 "" H 2400 3150 30  0000 C CNN
 	1    2400 3150
@@
 F 0 "R38" V 5800 6400 50  0000 C CNN
 F 1 "100R" V 5900 6400 50  0000 C CNN
-F 2 "CRF1:SMD-0603_r" H 5900 6400 60  0001 C CNN
+F 2 "Resistors_SMD:R_0805" H 5900 6400 60  0001 C CNN
 F 3 "" H 5900 6400 60  0001 C CNN
 	1    5900 6400
@@
 F 0 "D2" V 6000 6900 50  0000 C CNN
 F 1 "RED" V 5800 6950 50  0000 C CNN
-F 2 "LEDs:LED-0603" H 5900 6850 60  0001 C CNN
+F 2 "LEDs:LED_0805" H 5900 6850 60  0001 C CNN
 F 3 "" H 5900 6850 60  0001 C CNN
 	1    5900 6850
@@
 $EndComp
 $Comp
-L GND-RESCUE-BLDC_4 #PWR013
+L GND-RESCUE-BLDC_4 #PWR11
 U 1 1 53FC021C
 P 5900 7050
-F 0 "#PWR013" H 5900 7050 30  0001 C CNN
+F 0 "#PWR11" H 5900 7050 30  0001 C CNN
 F 1 "GND" H 5900 6980 30  0001 C CNN
 F 2 "" H 5900 7050 60  0001 C CNN
@@
 F 0 "R37" V 6100 6400 50  0000 C CNN
 F 1 "100R" V 6200 6400 50  0000 C CNN
-F 2 "CRF1:SMD-0603_r" H 6200 6400 60  0001 C CNN
+F 2 "Resistors_SMD:R_0805" H 6200 6400 60  0001 C CNN
 F 3 "" H 6200 6400 60  0001 C CNN
 	1    6200 6400
@@
 F 0 "D1" V 6300 6900 50  0000 C CNN
 F 1 "GREEN" V 6100 7000 50  0000 C CNN
-F 2 "LEDs:LED-0603" H 6200 6850 60  0001 C CNN
+F 2 "LEDs:LED_0805" H 6200 6850 60  0001 C CNN
 F 3 "" H 6200 6850 60  0001 C CNN
 	1    6200 6850
@@
 $EndComp
 $Comp
-L GND-RESCUE-BLDC_4 #PWR014
+L GND-RESCUE-BLDC_4 #PWR12
 U 1 1 53FC131A
 P 6200 7050
-F 0 "#PWR014" H 6200 7050 30  0001 C CNN
+F 0 "#PWR12" H 6200 7050 30  0001 C CNN
 F 1 "GND" H 6200 6980 30  0001 C CNN
 F 2 "" H 6200 7050 60  0001 C CNN
@@
 F 0 "D3" V 6600 6900 50  0000 C CNN
 F 1 "LED" V 6400 6950 50  0000 C CNN
-F 2 "LEDs:LED-0603" H 6500 6850 60  0001 C CNN
+F 2 "LEDs:LED_0805" H 6500 6850 60  0001 C CNN
 F 3 "" H 6500 6850 60  0001 C CNN
 	1    6500 6850
@@
 F 0 "R22" V 6400 6400 50  0000 C CNN
 F 1 "2k2" V 6500 6400 50  0000 C CNN
-F 2 "CRF1:SMD-0603_r" H 6500 6400 60  0001 C CNN
+F 2 "Resistors_SMD:R_0805" H 6500 6400 60  0001 C CNN
 F 3 "" H 6500 6400 60  0001 C CNN
 	1    6500 6400
@@
 $EndComp
 $Comp
-L GND-RESCUE-BLDC_4 #PWR015
+L GND-RESCUE-BLDC_4 #PWR14
 U 1 1 53FC8AA4
 P 6500 7050
-F 0 "#PWR015" H 6500 7050 30  0001 C CNN
+F 0 "#PWR14" H 6500 7050 30  0001 C CNN
 F 1 "GND" H 6500 6980 30  0001 C CNN
 F 2 "" H 6500 7050 60  0001 C CNN
@@
 $EndComp
 $Comp
-L VCC #PWR016
+L VCC #PWR13
 U 1 1 53FC98D2
 P 6500 6150
-F 0 "#PWR016" H 6500 6250 30  0001 C CNN
+F 0 "#PWR13" H 6500 6250 30  0001 C CNN
 F 1 "VCC" V 6500 6300 30  0000 C CNN
 F 2 "" H 6500 6150 60  0001 C CNN
@@
 $Bitmap
 Pos 9900 5750
-Scale 0,000000
+Scale 0.000000
 Data
 89 50 4E 47 0D 0A 1A 0A 00 00 00 0D 49 48 44 52 00 00 03 4C 00 00 02 2D 08 02 00 00 00 85 20 6D
@@
 20 08 82 20 08 12 3C 28 79 08 82 20 08 82 20 2D 08 4A 1E 82 20 08 82 20 48 0B 82 92 87 20 08 82
 20 08 D2 82 A0 E4 21 08 82 20 08 82 B4 20 28 79 08 82 20 08 82 20 2D 08 4A 1E 82 20 08 82 20 48
-0B F2 FF 19 12 7F 86 40 CA 02 9D 00 00 00 00 49 45 4E 44 AE 42 60 82 00
+0B F2 FF 19 12 7F 86 40 CA 02 9D 00 00 00 00 49 45 4E 44 AE 42 60 82
 EndData
 $EndBitmap
@@
 $EndComp
 $Comp
-L +5V #PWR017
+L +5V #PWR1
 U 1 1 54036995
 P 1450 3750
-F 0 "#PWR017" H 1450 3840 20  0001 C CNN
+F 0 "#PWR1" H 1450 3840 20  0001 C CNN
 F 1 "+5V" H 1450 3840 30  0000 C CNN
 F 2 "" H 1450 3750 60  0001 C CNN
@@
 $EndComp
 $Comp
-L GND-RESCUE-BLDC_4 #PWR018
+L GND-RESCUE-BLDC_4 #PWR22
 U 1 1 548F24DF
 P 9850 5050
-F 0 "#PWR018" H 9850 5050 30  0001 C CNN
+F 0 "#PWR22" H 9850 5050 30  0001 C CNN
 F 1 "GND" H 9850 4980 30  0001 C CNN
 F 2 "" H 9850 5050 60  0001 C CNN
@@
 $EndComp
 $Comp
-L GND-RESCUE-BLDC_4 #PWR019
+L GND-RESCUE-BLDC_4 #PWR19
 U 1 1 548F2504
 P 8450 5100
-F 0 "#PWR019" H 8450 5100 30  0001 C CNN
+F 0 "#PWR19" H 8450 5100 30  0001 C CNN
 F 1 "GND" H 8450 5030 30  0001 C CNN
 F 2 "" H 8450 5100 60  0001 C CNN
@@
 $EndComp
 $Comp
-L GND-RESCUE-BLDC_4 #PWR020
+L GND-RESCUE-BLDC_4 #PWR17
 U 1 1 548F2529
 P 8150 4600
-F 0 "#PWR020" H 8150 4600 30  0001 C CNN
+F 0 "#PWR17" H 8150 4600 30  0001 C CNN
 F 1 "GND" H 8150 4530 30  0001 C CNN
 F 2 "" H 8150 4600 60  0001 C CNN
@@
 $EndComp
 $Comp
-L GND-RESCUE-BLDC_4 #PWR021
+L GND-RESCUE-BLDC_4 #PWR18
 U 1 1 548F254E
 P 8300 4100
-F 0 "#PWR021" H 8300 4100 30  0001 C CNN
+F 0 "#PWR18" H 8300 4100 30  0001 C CNN
 F 1 "GND" H 8300 4030 30  0001 C CNN
 F 2 "" H 8300 4100 60  0001 C CNN
@@
 $EndComp
 $Comp
-L GND-RESCUE-BLDC_4 #PWR022
+L GND-RESCUE-BLDC_4 #PWR20
 U 1 1 548F2573
 P 9100 1500
-F 0 "#PWR022" H 9100 1500 30  0001 C CNN
+F 0 "#PWR20" H 9100 1500 30  0001 C CNN
 F 1 "GND" H 9100 1430 30  0001 C CNN
 F 2 "" H 9100 1500 60  0001 C CNN
