File: Projects/VESC/design/Power.sch (KiCad schematic (older format))
At the start: 48 parts, among them U2 TC2117, U3 DRV8302

Commit message: Started making changes to VESC layout and schematic
Parts:
- C18, C19, C20, C21, C22, C23, C24, C26, C27, C28, C29, C30, C34, C36, C52: footprint CRF1:SMD-0603_c -> Capacitors_SMD:C_0805
- R17, R18, R19, R20, R21, R23, R24, R25, R26, R27, R32, R33, R48, R49, R50, R51: footprint CRF1:SMD-0603_r -> Resistors_SMD:R_0805
- U2: symbol NCP1117ST33T3G -> NCP1117ST33T3G-RESCUE-BLDC_4
Connections:
- net +5V: now also U2.3 (VI)
- net GND: now also U2.1 (GND)
- net VCC: now also U2.2 (VO)
Other:
- moved on the sheet: U2
