File: Projects/VESC/design/temp.sch (KiCad schematic (older format))
At the start: 3 parts

Commit message: Started making changes to VESC layout and schematic
Parts:
- C41: footprint CRF1:SMD-0603_c -> Capacitors_SMD:C_0805
- R1, R2: footprint CRF1:SMD-0603_r -> Resistors_SMD:R_0805
Changed lines of the file:
@@
 F 0 "R1" V 4480 3400 40  0000 C CNN
 F 1 "NTC 10k" V 4407 3401 40  0000 C CNN
-F 2 "CRF1:SMD-0603_r" V 4330 3400 30  0001 C CNN
+F 2 "Resistors_SMD:R_0805" V 4330 3400 30  0001 C CNN
 F 3 "" H 4400 3400 30  0000 C CNN
 	1    4400 3400
@@
 F 0 "R2" V 4480 4100 40  0000 C CNN
 F 1 "10k" V 4407 4101 40  0000 C CNN
-F 2 "CRF1:SMD-0603_r" V 4330 4100 30  0001 C CNN
+F 2 "Resistors_SMD:R_0805" V 4330 4100 30  0001 C CNN
 F 3 "" H 4400 4100 30  0000 C CNN
 	1    4400 4100
@@
 F 0 "C41" H 4150 4200 40  0000 L CNN
 F 1 "2.2u" H 4156 4015 40  0000 L CNN
-F 2 "CRF1:SMD-0603_c" H 4188 3950 30  0001 C CNN
+F 2 "Capacitors_SMD:C_0805" H 4188 3950 30  0001 C CNN
 F 3 "" H 4150 4100 60  0000 C CNN
 	1    4150 4100
@@
 $EndComp
 $Comp
-L VCC #PWR023
+L VCC #PWR23
 U 1 1 5426DB11
 P 4400 3050
-F 0 "#PWR023" H 4400 3150 30  0001 C CNN
+F 0 "#PWR23" H 4400 3150 30  0001 C CNN
 F 1 "VCC" H 4400 3150 30  0000 C CNN
 F 2 "" H 4400 3050 60  0000 C CNN
@@
 $EndComp
 $Comp
-L GND-RESCUE-BLDC_4 #PWR024
+L GND-RESCUE-BLDC_4 #PWR24
 U 1 1 5426DB25
 P 4400 4600
-F 0 "#PWR024" H 4400 4600 30  0001 C CNN
+F 0 "#PWR24" H 4400 4600 30  0001 C CNN
 F 1 "GND" H 4400 4530 30  0001 C CNN
 F 2 "" H 4400 4600 60  0000 C CNN
