File: Projects/KiCad_USB/RH025.1.sch (KiCad schematic (older format))
At the start: 27 parts, among them IC1 FE1.1S, J1 POWER_JACKCOMBO

Commit message: Started work on cleaning up FE1.1s USB hub and VESC backplane
Parts:
- removed IC1: FE1.1S, RH025.1:FE1.1S_SSOP-28, symbol FE1.1S
- removed J1: POWER_JACKCOMBO, RH025.1:POWER_JACK_COMBO, symbol POWER_JACKCOMBO
- removed SV1: ~, RH025.1:MA04-1, symbol MA04-1
- removed USB5: USBA-PTH, RH025.1:USB-A-F-PTH, symbol USBA-PTH
- added M?: FE1.1S, FE1.1S_SSOP-28, symbol FE1.1S
- added USB?: USBA-PTH, USB-A-F-PTH, symbol USBA-PTH
- ACT7, PORT1, PORT2, PORT3, PORT4: footprint RH025.1:LED-0603 -> LEDs:LED_0805
- C1, C2, C3, C4, C5, C6: footprint RH025.1:CAP-0603 -> Capacitors_SMD:C_0805
- R1, R2, R3, R4, R5, REXT7: footprint RH025.1:RES-0603 -> Resistors_SMD:R_0805
Connections:
- wire segments 112 -> 106
Other:
- note removed: "0x60"
- note removed: "0xC0"
- note removed: "0xC1"
- note removed: "7-bit I2C Address is 0x40"
- note removed: "CLEAR BOTH SIDES OF SJ1"
- note removed: "I2C read is 0x81"
- note removed: "I2C write is 0x80"
- note removed: "Read Address:"
- note removed: "Slave Address:"
- note removed: "TO DISABLE I2C PULLUP RESISTORS"
- note removed: "VCC = 3.6V Max"
- note removed: "Write Address:"
Changed lines of the file:
@@
 EESchema Schematic File Version 2
 LIBS:RH025.1
+LIBS:USST-parts
+LIBS:RH025.1-cache
 EELAYER 25 0
 EELAYER END
@@
 Comment4 ""
 $EndDescr
-Text Notes 12950 4050 0    70   ~ 0
-CLEAR BOTH SIDES OF SJ1
-Text Notes 12950 4150 0    70   ~ 0
-TO DISABLE I2C PULLUP RESISTORS
-Text Notes 10750 5950 0    70   ~ 0
-7-bit I2C Address is 0x40
-Text Notes 10750 6050 0    70   ~ 0
-I2C write is 0x80
-Text Notes 10750 6150 0    70   ~ 0
-I2C read is 0x81
-Text Notes 11550 7950 0    70   ~ 0
-VCC = 3.6V Max
-Text Notes 11550 8150 0    70   ~ 0
-Read Address:
-Text Notes 11550 8250 0    70   ~ 0
-Write Address:
-Text Notes 11550 8050 0    70   ~ 0
-Slave Address:
-Text Notes 12450 8050 0    70   ~ 0
-0x60
-Text Notes 12450 8150 0    70   ~ 0
-0xC1
-Text Notes 12450 8250 0    70   ~ 0
-0xC0
 $Comp
 L LED0603 ACT7
@@
 F 0 "ACT7" V 7625 4625 60  0000 L BNN
 F 1 "~" H 7640 4490 65  0001 L TNN
-F 2 "RH025.1:LED-0603" H 7640 4390 65  0001 L TNN
+F 2 "LEDs:LED_0805" H 7640 4390 65  0001 L TNN
 F 3 "" H 7650 4600 60  0001 C CNN
 	1    7650 4600
@@
 F 0 "C1" V 4835 6410 60  0000 L BNN
 F 1 "0.1uF" V 4925 6665 60  0000 L BNN
-F 2 "RH025.1:CAP-0603" H 4840 6390 65  0001 L TNN
+F 2 "Capacitors_SMD:C_0805" H 4840 6390 65  0001 L TNN
 F 3 "" H 4850 6600 60  0001 C CNN
 	1    4850 6600
@@
 F 0 "C2" V 4635 6410 60  0000 L BNN
 F 1 "10uF" V 4725 6665 60  0000 L BNN
-F 2 "RH025.1:CAP-0603" H 4640 6390 65  0001 L TNN
+F 2 "Capacitors_SMD:C_0805" H 4640 6390 65  0001 L TNN
 F 3 "" H 4650 6600 60  0001 C CNN
 	1    4650 6600
@@
 F 0 "C3" V 4435 6410 60  0000 L BNN
 F 1 "0.1uF" V 4525 6665 60  0000 L BNN
-F 2 "RH025.1:CAP-0603" H 4440 6390 65  0001 L TNN
+F 2 "Capacitors_SMD:C_0805" H 4440 6390 65  0001 L TNN
 F 3 "" H 4450 6600 60  0001 C CNN
 	1    4450 6600
@@
 F 0 "C4" V 4235 6410 60  0000 L BNN
 F 1 "10uF" V 4325 6665 60  0000 L BNN
-F 2 "RH025.1:CAP-0603" H 4240 6390 65  0001 L TNN
+F 2 "Capacitors_SMD:C_0805" H 4240 6390 65  0001 L TNN
 F 3 "" H 4250 6600 60  0001 C CNN
 	1    4250 6600
 	1    0    0    -1
-$EndComp
-$Comp
-L CAP0603 C5
-U 1 1 57E6C997
-P 4400 4550
-F 0 "C5" V 4386 4360 60  0000 L BNN
-F 1 "10uF" V 4474 4615 60  0000 L BNN
-F 2 "RH025.1:CAP-0603" H 4390 4340 65  0001 L TNN
-F 3 "" H 4400 4550 60  0001 C CNN
-	1    4400 4550
-	0    1    1    0
-$EndComp
-$Comp
-L CAP0603 C6
-U 1 1 57E6CA5F
-P 4400 4750
-F 0 "C6" V 4386 4560 60  0000 L BNN
-F 1 "0.1uF" V 4474 4815 60  0000 L BNN
-F 2 "RH025.1:CAP-0603" H 4390 4540 65  0001 L TNN
-F 3 "" H 4400 4750 60  0001 C CNN
-	1    4400 4750
-	0    1    1    0
 $EndComp
 $Comp
@@
 P 5550 8450
 F 0 "#GND01" H 5450 8450 60  0001 L BNN
-F 1 "GND" H 5450 8450 60  0000 L BNN
+F 1 "GND" H 5600 8500 60  0000 L BNN
 F 2 "" H 5550 8450 60  0001 C CNN
 F 3 "" H 5550 8450 60  0001 C CNN
@@
 F 3 "" H 7650 5450 60  0001 C CNN
 	1    7650 5450
-	1    0    0    -1
-$EndComp
-$Comp
-L FE1.1S IC1
-U 1 1 57E6CD1B
-P 5900 5550
-F 0 "IC1" H 5501 6780 60  0000 L BNN
-F 1 "FE1.1S" H 5890 5440 65  0001 L TNN
-F 2 "RH025.1:FE1.1S_SSOP-28" H 5890 5340 65  0001 L TNN
-F 3 "" H 5900 5550 60  0001 C CNN
-	1    5900 5550
-	1    0    0    -1
-$EndComp
-$Comp
-L POWER_JACKCOMBO J1
-U 1 1 57E6CDE3
-P 9200 5900
-F 0 "J1" H 8800 5900 70  0000 L BNN
-F 1 "POWER_JACKCOMBO" H 8800 6300 70  0000 L BNN
-F 2 "RH025.1:POWER_JACK_COMBO" H 9190 5690 65  0001 L TNN
-F 3 "" H 9200 5900 60  0001 C CNN
-	1    9200 5900
 	1    0    0    -1
 $EndComp
@@
 F 0 "PORT1" V 7326 4150 60  0000 L BNN
 F 1 "~" V 7425 4250 60  0000 L BNN
-F 2 "RH025.1:LED-0603" H 7340 4340 65  0001 L TNN
+F 2 "LEDs:LED_0805" H 7340 4340 65  0001 L TNN
 F 3 "" H 7350 4550 60  0001 C CNN
 	1    7350 4550
@@
 F 0 "PORT2" V 7301 4550 60  0000 L BNN
 F 1 "~" V 7425 4650 60  0000 L BNN
-F 2 "RH025.1:LED-0603" H 7340 4740 65  0001 L TNN
+F 2 "LEDs:LED_0805" H 7340 4740 65  0001 L TNN
 F 3 "" H 7350 4950 60  0001 C CNN
 	1    7350 4950
@@
 F 0 "PORT3" V 7225 4675 60  0000 L BNN
 F 1 "~" H 7240 4540 65  0001 L TNN
-F 2 "RH025.1:LED-0603" H 7240 4440 65  0001 L TNN
+F 2 "LEDs:LED_0805" H 7240 4440 65  0001 L TNN
 F 3 "" H 7250 4650 60  0001 C CNN
 	1    7250 4650
@@
 F 0 "PORT4" V 7225 5075 60  0000 L BNN
 F 1 "~" H 7240 4940 65  0001 L TNN
-F 2 "RH025.1:LED-0603" H 7240 4840 65  0001 L TNN
+F 2 "LEDs:LED_0805" H 7240 4840 65  0001 L TNN
 F 3 "" H 7250 5050 60  0001 C CNN
 	1    7250 5050
@@
 F 0 "R1" H 4195 5560 60  0000 L BNN
 F 1 "100K" H 4500 5475 60  0000 L BNN
-F 2 "RH025.1:RES-0603" H 4390 5340 65  0001 L TNN
+F 2 "Resistors_SMD:R_0805" H 4390 5340 65  0001 L TNN
 F 3 "" H 4400 5550 60  0001 C CNN
 	1    4400 5550
@@
 F 0 "R2" H 4495 5160 60  0000 L BNN
 F 1 "47K" H 4800 5075 60  0000 L BNN
-F 2 "RH025.1:RES-0603" H 4690 4940 65  0001 L TNN
+F 2 "Resistors_SMD:R_0805" H 4690 4940 65  0001 L TNN
 F 3 "" H 4700 5150 60  0001 C CNN
 	1    4700 5150
@@
 F 0 "R3" H 6645 4609 60  0000 L BNN
 F 1 "330" H 6625 4525 60  0000 L BNN
-F 2 "RH025.1:RES-0603" H 6840 4390 65  0001 L TNN
+F 2 "Resistors_SMD:R_0805" H 6840 4390 65  0001 L TNN
 F 3 "" H 6850 4600 60  0001 C CNN
 	1    6850 4600
@@
 F 0 "R4" H 6645 5009 60  0000 L BNN
 F 1 "330" H 6625 4925 60  0000 L BNN
-F 2 "RH025.1:RES-0603" H 6840 4790 65  0001 L TNN
+F 2 "Resistors_SMD:R_0805" H 6840 4790 65  0001 L TNN
 F 3 "" H 6850 5000 60  0001 C CNN
 	1    6850 5000
@@
 F 0 "R5" H 7445 5060 60  0000 L BNN
 F 1 "330" H 7750 4975 60  0000 L BNN
-F 2 "RH025.1:RES-0603" H 7640 4840 65  0001 L TNN
+F 2 "Resistors_SMD:R_0805" H 7640 4840 65  0001 L TNN
 F 3 "" H 7650 5050 60  0001 C CNN
 	1    7650 5050
@@
 F 0 "REXT7" H 4345 5860 60  0000 L BNN
 F 1 "2.7K" H 4650 5775 60  0000 L BNN
-F 2 "RH025.1:RES-0603" H 4540 5640 65  0001 L TNN
+F 2 "Resistors_SMD:R_0805" H 4540 5640 65  0001 L TNN
 F 3 "" H 4550 5850 60  0001 C CNN
 	1    4550 5850
-	1    0    0    -1
-$EndComp
-$Comp
-L MA04-1 SV1
-U 1 1 57E6D7A7
-P 8600 4700
-F 0 "SV1" H 8551 4930 70  0000 L BNN
-F 1 "~" H 8590 4590 65  0001 L TNN
-F 2 "RH025.1:MA04-1" H 8590 4490 65  0001 L TNN
-F 3 "" H 8600 4700 60  0001 C CNN
-	1    8600 4700
 	1    0    0    -1
 $EndComp
@@
 P 5250 4300
 F 0 "#U$05" H 5175 4400 60  0001 L BNN
-F 1 "VBUS" H 5175 4400 60  0000 L BNN
+F 1 "VBUS" H 5150 4500 60  0000 L BNN
 F 2 "" H 5250 4300 60  0001 C CNN
 F 3 "" H 5250 4300 60  0001 C CNN
@@
 P 5700 7250
 F 0 "#U$06" H 5625 7350 60  0001 L BNN
-F 1 "VBUS" H 5625 7350 60  0000 L BNN
+F 1 "VBUS" H 5600 7450 60  0000 L BNN
 F 2 "" H 5700 7250 60  0001 C CNN
 F 3 "" H 5700 7250 60  0001 C CNN
@@
 P 4850 5350
 F 0 "#U$08" H 4775 5450 60  0001 L BNN
-F 1 "3V3" H 4775 5450 60  0000 L BNN
+F 1 "3V3" H 4800 5550 60  0000 L BNN
 F 2 "" H 4850 5350 60  0001 C CNN
 F 3 "" H 4850 5350 60  0001 C CNN
@@
 $EndComp
 $Comp
-L USBA-PTH USB5
-U 1 1 57E6DD1F
-P 6800 5300
-F 0 "USB5" H 6790 5290 65  0001 L TNN
-F 1 "USBA-PTH" H 6790 5190 65  0001 L TNN
-F 2 "RH025.1:USB-A-F-PTH" H 6790 5090 65  0001 L TNN
-F 3 "" H 6800 5300 60  0001 C CNN
-	1    6800 5300
-	0    1    -1   0
-$EndComp
-$Comp
 L CRYSTALHC49UP XL1
 U 1 1 57E6DDE7
 P 5100 4800
-F 0 "XL1" H 4880 4815 60  0000 L BNN
-F 1 "12MHz" H 5180 4725 60  0000 L BNN
+F 0 "XL1" H 5050 4550 60  0000 L BNN
+F 1 "12MHz" H 4950 4650 60  0000 L BNN
 F 2 "RH025.1:HC49UP" H 5090 4590 65  0001 L TNN
 F 3 "" H 5100 4800 60  0001 C CNN
@@
 Connection ~ 4850 5450
 Wire Wire Line
-	8900 4700 9400 4700
-Text Label 9200 4700 0    65   ~ 0
-D+
-Wire Wire Line
 	5300 6650 5300 7700
 Wire Wire Line
@@
 Wire Wire Line
 	5200 6550 5300 6550
-Wire Wire Line
-	8900 4600 9400 4600
-Text Label 9200 4600 0    65   ~ 0
-D-
 Wire Wire Line
 	4850 6850 4850 6800
@@
 	7650 5350 7650 5250
 Wire Wire Line
-	8900 4800 9400 4800
-Text Label 9200 4800 0    65   ~ 0
-GND
-Wire Wire Line
-	9300 5800 9700 5800
-Text Label 9500 5800 0    65   ~ 0
-GND
-Wire Wire Line
 	5550 8350 5550 8100
 Wire Wire Line
@@
 Connection ~ 7350 6750
 Connection ~ 8150 6750
-Wire Wire Line
-	8900 4900 9400 4900
-Text Label 9200 4900 0    65   ~ 0
-VBUS
-Wire Wire Line
-	9300 5600 9700 5600
-Text Label 9500 5600 0    65   ~ 0
-VBUS
 Text Label 5300 5450 2    10   ~ 0
 3V3
@@
 Text Label 5300 5650 2    10   ~ 0
 3V3
-Text Label 8900 4700 0    10   ~ 0
-D+
 Text Label 5300 6650 2    10   ~ 0
 D+
@@
 Text Label 4850 7600 0    10   ~ 0
 D-
-Text Label 8900 4600 0    10   ~ 0
-D-
 Text GLabel 4550 6900 1    10   UnSpc ~ 0
 GND
@@
 GND
 Text GLabel 7650 5350 1    10   UnSpc ~ 0
-GND
-Text GLabel 8900 4800 2    10   UnSpc ~ 0
-GND
-Text GLabel 9300 5800 2    10   UnSpc ~ 0
 GND
 Text GLabel 5550 8350 1    10   UnSpc ~ 0
@@
 Text Label 8300 6350 3    10   ~ 0
 VBUS
-Text Label 8900 4900 0    10   ~ 0
-VBUS
-Text Label 9300 5600 0    10   ~ 0
-VBUS
+$Comp
+L FE1.1S M?
+U 1 1 5862FDC9
+P 5900 5550
+F 0 "M?" H 5500 6780 45  0000 L BNN
+F 1 "FE1.1S" H 5900 5550 45  0001 L BNN
+F 2 "FE1.1S_SSOP-28" H 5930 5700 20  0001 C CNN
+F 3 "" H 5900 5550 60  0001 C CNN
+	1    5900 5550
+	1    0    0    -1
+$EndComp
+$Comp
+L CAP0603 C5
+U 1 1 57E6C997
+P 4400 4550
+F 0 "C5" V 4386 4360 60  0000 L BNN
+F 1 "10uF" V 4474 4615 60  0000 L BNN
+F 2 "Capacitors_SMD:C_0805" H 4390 4340 65  0001 L TNN
+F 3 "" H 4400 4550 60  0001 C CNN
+	1    4400 4550
+	0    1    1    0
+$EndComp
+$Comp
+L CAP0603 C6
+U 1 1 57E6CA5F
+P 4400 4750
+F 0 "C6" V 4386 4560 60  0000 L BNN
+F 1 "0.1uF" V 4474 4815 60  0000 L BNN
+F 2 "Capacitors_SMD:C_0805" H 4390 4540 65  0001 L TNN
+F 3 "" H 4400 4750 60  0001 C CNN
+	1    4400 4750
+	0    1    1    0
+$EndComp
+$Comp
+L USBA-PTH USB?
+U 1 1 5863183A
+P 6800 5300
+F 0 "USB?" H 6800 5300 45  0001 C CNN
+F 1 "USBA-PTH" H 6800 5300 45  0001 C CNN
+F 2 "USB-A-F-PTH" H 6830 5450 20  0001 C CNN
+F 3 "" H 6800 5300 60  0001 C CNN
+	1    6800 5300
+	0    -1   -1   0
+$EndComp
 $EndSCHEMATC

Commit message: Further cleanup of Fe1.1s schematic
Parts:
- removed USB1: USBMICROB-PTH, RH025.1:USB-MICROB-TH, symbol USBMICROB-PTH
- removed USB2, USB3, USB4: USBA-PTH, RH025.1:USB-A-F-PTH, symbol USBA-PTH
- removed USB?: USBA-PTH, USB-A-F-PTH, symbol USBA-PTH
- added USB? (x5): USB-TYPA, USB-A-F-PTH, symbol USB-TYPA
- PORT1, PORT2, PORT3, PORT4: symbol LED0603 -> LED_SMT
- XL1: symbol CRYSTALHC49UP -> XTAL_1
Connections:
- net D+: now also USB?.D+
- net D-: now also USB?.D-
- net GND: now also USB?.GND, USB?.GND, USB?.GND, USB?.GND; no longer R5.1
- net N$11: now also USB?.D+
- net N$12: now also USB?.D-
- net N$14: now also USB?.D+
- net N$15: now also USB?.D-
- net N$16: now also USB?.D+
- net N$17: now also USB?.D-
- net N$18: now also USB?.D+
- net N$19: now also USB?.D-
- net N$3: now also USB?.VBUS
- net N$4: now also USB?.GND
- net VBUS: now also USB?.VBUS, USB?.VBUS, USB?.VBUS, USB?.VBUS

Commit message: Changed a part as demonstration
Parts:
- ACT7: symbol LED0603 -> LED_SMT
- R3: symbol RES0603 -> R
Changed lines of the file:
@@
 $EndDescr
 $Comp
-L LED0603 ACT7
+L LED_SMT ACT7
 U 1 1 57E6C5AF
-P 7650 4600
-F 0 "ACT7" V 7625 4625 60  0000 L BNN
-F 1 "~" H 7640 4490 65  0001 L TNN
-F 2 "LEDs:LED_0805" H 7640 4390 65  0001 L TNN
-F 3 "" H 7650 4600 60  0001 C CNN
-	1    7650 4600
-	-1   0    0    -1
+P 7650 4700
+F 0 "ACT7" V 7750 4850 60  0000 L BNN
+F 1 "~" H 7640 4590 65  0001 L TNN
+F 2 "LEDs:LED_0805" H 7640 4490 65  0001 L TNN
+F 3 "" H 7650 4700 60  0001 C CNN
+	1    7650 4700
+	0    1    -1   0
 $EndComp
 $Comp
@@
 $EndComp
 $Comp
-L RES0603 R3
+L R R3
 U 1 1 57E6D487
 P 6850 4600
-F 0 "R3" H 6645 4609 60  0000 L BNN
-F 1 "330" H 6625 4525 60  0000 L BNN
+F 0 "R3" V 6800 4600 60  0000 L BNN
+F 1 "330" V 7000 4550 60  0000 L BNN
 F 2 "Resistors_SMD:R_0805" H 6840 4390 65  0001 L TNN
 F 3 "" H 6850 4600 60  0001 C CNN
 	1    6850 4600
-	1    0    0    1
+	0    -1   1    0
 $EndComp
 $Comp
@@
 	5300 5150 5250 5150
 Wire Wire Line
-	5250 5150 5250 5450
-Wire Wire Line
-	5250 5450 5250 5650
-Wire Wire Line
-	4850 5450 5250 5450
-Wire Wire Line
-	5250 5450 5300 5450
-Wire Wire Line
-	4850 5350 4850 5450
-Wire Wire Line
-	4850 5450 4850 6250
-Wire Wire Line
-	4650 6250 4850 6250
-Wire Wire Line
-	4850 6250 5250 6250
-Wire Wire Line
-	5250 6250 5300 6250
-Wire Wire Line
-	4850 6350 5250 6350
-Wire Wire Line
-	5250 6350 5300 6350
+	5250 5150 5250 5650
+Wire Wire Line
+	4850 5450 5300 5450
+Wire Wire Line
+	4850 5350 4850 6250
+Wire Wire Line
+	4650 6250 5300 6250
+Wire Wire Line
+	4850 6350 5300 6350
 Wire Wire Line
 	5250 6350 5250 6250
@@
 	4850 6850 4850 6800
 Wire Wire Line
-	4100 6850 4250 6850
-Wire Wire Line
-	4250 6850 4450 6850
-Wire Wire Line
-	4450 6850 4550 6850
-Wire Wire Line
-	4550 6850 4650 6850
-Wire Wire Line
-	4650 6850 4850 6850
+	4100 6850 4850 6850
 Wire Wire Line
 	4550 6850 4550 6900
@@
 	4250 6800 4250 6850
 Wire Wire Line
-	4350 5850 4100 5850
-Wire Wire Line
-	4100 4450 4100 4550
-Wire Wire Line
-	4100 4550 4100 4750
-Wire Wire Line
-	4100 4750 4100 5550
-Wire Wire Line
-	4100 5550 4100 5850
-Wire Wire Line
-	4100 5850 4100 6850
+	4100 5850 4350 5850
+Wire Wire Line
+	4100 4450 4100 6850
 Wire Wire Line
 	5300 4450 4100 4450
@@
 Connection ~ 4650 6850
 Wire Wire Line
-	6650 5550 6650 6850
-Wire Wire Line
-	6650 6850 6650 6950
+	6650 5550 6650 6950
 Wire Wire Line
 	7050 5850 7050 6850
 Wire Wire Line
-	6650 6850 7050 6850
-Wire Wire Line
-	7050 6850 7450 6850
-Wire Wire Line
-	7450 6850 7850 6850
+	6650 6850 7850 6850
 Wire Wire Line
 	7450 6850 7450 6150
@@
 	7050 5000 7100 5000
 Wire Wire Line
-	7100 4950 7100 5000
-Wire Wire Line
-	7100 5000 7100 5050
+	7100 4950 7100 5050
 Wire Wire Line
 	7100 4950 7150 4950
@@
 	5250 4750 5300 4750
 Wire Wire Line
-	4950 6050 5250 6050
-Wire Wire Line
-	5250 6050 5300 6050
-Wire Wire Line
-	4450 6150 5250 6150
-Wire Wire Line
-	5250 6150 5300 6150
+	4950 6050 5300 6050
+Wire Wire Line
+	4450 6150 5300 6150
 Wire Wire Line
 	5250 6150 5250 6050
@@
 	6850 5750 6850 5550
 Wire Wire Line
-	4600 5550 4700 5550
-Wire Wire Line
-	4700 5550 5300 5550
+	4600 5550 5300 5550
 Wire Wire Line
 	4700 5550 4700 5350
@@
 	8050 6650 8050 6450
 Wire Wire Line
-	7050 4600 7100 4600
-Wire Wire Line
-	7100 4550 7100 4600
-Wire Wire Line
-	7100 4600 7100 4650
+	7000 4600 7100 4600
+Wire Wire Line
+	7100 4550 7100 4650
 Wire Wire Line
 	7100 4550 7150 4550
@@
 	6600 4550 6600 4600
 Wire Wire Line
-	6600 4600 6650 4600
+	6600 4600 6700 4600
 Wire Wire Line
 	6500 4650 6600 4650
@@
 	7450 4550 7500 4550
 Wire Wire Line
-	7500 4450 7500 4550
-Wire Wire Line
-	7500 4550 7500 4650
-Wire Wire Line
-	7500 4650 7500 4950
-Wire Wire Line
-	7500 4950 7500 5050
+	7500 4450 7500 5050
 Wire Wire Line
 	7500 4950 7450 4950
@@
 	7500 5050 7450 5050
 Wire Wire Line
-	6500 4450 7500 4450
-Wire Wire Line
-	7500 4450 7650 4450
+	6500 4450 7650 4450
 Wire Wire Line
 	7650 4450 7650 4500
@@
 Connection ~ 7500 4450
 Wire Wire Line
-	4600 4550 4700 4550
-Wire Wire Line
-	4700 4550 5250 4550
-Wire Wire Line
-	5250 4550 5300 4550
+	4600 4550 5300 4550
 Wire Wire Line
 	5250 4550 5250 4300
 Wire Wire Line
-	4700 4550 4700 4750
-Wire Wire Line
-	4700 4750 4700 4950
+	4700 4550 4700 4950
 Wire Wire Line
 	4600 4750 4700 4750
@@
 	8150 6750 8150 6450
 Wire Wire Line
-	7750 6150 7750 6750
-Wire Wire Line
-	6950 6750 7350 6750
-Wire Wire Line
-	7350 6750 7750 6750
-Wire Wire Line
-	7750 6750 8150 6750
-Wire Wire Line
-	8150 6750 8450 6750
+	7750 6750 7750 6150
+Wire Wire Line
+	6950 6750 8450 6750
 Wire Wire Line
 	7350 5850 7350 6750

Commit message: Generalizing Kicad symbols
Parts:
- C1, C2, C3, C4, C5, C6: symbol CAP0603 -> C
- R1, R2, R4, R5, REXT7: symbol RES0603 -> R
Connections:
- net GND: now also R1.2, R5.2; no longer R1.1
- net N$13: now also R1.1, R2.2; no longer R1.2, R2.1
- net N$22: now also R5.1; no longer R5.2
- net VBUS renamed +5V
- net +5V: now also R2.1; no longer R2.2
