File: Projects/USSTCM/USSTCM.kicad_pcb (KiCad board)
At the start: 4 copper layers, 99.1 x 40.6 mm, 108 parts, among them IC1 REG1117, IC2 REG1117, IC3 RASPI_LAN9514, IC5 FSUSB42MSOP10, Q1 DMG1012T, Q2 DMG1012T, Q3 DMG1012T, Q4 DMG1012T, Q6 CTS_32X25_SMD, U1 RASPI, U2 MCP2515, U3 AMIS-42770, U4 AMIS-42770, U5 AMIS-42770, U6 AMIS-42770, U7 MCP2562

Commit message: added differential routes
Parts:
- removed ACT55: ~, USSTCM:LED_CHIP-LED0603
- removed CAM0: FFC-15, USSTCM:RASPI_FFC-15
- removed D6: BAV99, USSTCM:DIODE_SOT23
- removed ETHERNET55: HR911105A, USSTCM:HANRUN_RJ45
- removed GPIO55: PI_GPIO, USSTCM2:RASPI_RASPI_GPIO_B+_PIN
- removed HDMI55: HDMI, USSTCM:RASPI_HDMI
- removed Q6: CTS_32X25_SMD, USSTCM:RASPI_CTS_32X25
- removed U3, U4, U5, U6: AMIS-42770, Housings_SOIC:SOIC-20_7.5x12.8mm_Pitch1.27mm
- removed U7: MCP2562, Housings_SOIC:SOIC-8_3.9x4.9mm_Pitch1.27mm
- removed USB55: USB2, USSTCM:RASPI_USB2
- added ACT1: ~, LEDs:LED_0805, F.Cu at (134.4, 49.2)
- added C3: 10u, Capacitors_SMD:C_0805, F.Cu at (168.7, 46.6)
- added C47: 10u, Capacitors_SMD:C_0805, F.Cu at (193.3, 148.4)
- added C48: 10u, Capacitors_SMD:C_0805, F.Cu at (178.9, 160.8)
- added C5: 20p, Capacitors_SMD:C_0805, F.Cu at (27.2, 162.2)
- added C50: 10u, Capacitors_SMD:C_0805, F.Cu at (229.5, 19.8)
- added C51: 0.01u, Capacitors_SMD:C_0805, F.Cu at (233.7, 19.8)
- added C52: 0.01u, Capacitors_SMD:C_0805, F.Cu at (230.5, 25.0)
- added C53: 100n, Capacitors_SMD:C_0805, F.Cu at (226.2, 30.3)
- added C54: 100n, Capacitors_SMD:C_0805, F.Cu at (238.0, 19.6)
- added C55: 100n, Capacitors_SMD:C_0805, F.Cu at (230.2, 30.2)
- added C56: 100n, Capacitors_SMD:C_0805, F.Cu at (237.3, 14.4)
- added C57: 100n, Capacitors_SMD:C_0805, F.Cu at (226.2, 25.1)
- added CAM2: RASPI_CAM, USST-footprints:FFC-15-PICAM, F.Cu at (204.4, 50.8)
- added D1: BAV99, USSTCM:DIODE_SOT23, F.Cu at (269.5, -37.5)
- added FB3: 80mA Ferrite, Capacitors_SMD:C_0805, F.Cu at (219.1, 25.8)
- added HDMI1: HDMI, USSTCM:RASPI_HDMI, F.Cu at (256.7, -41.0)
- added IC4: REG1117, USSTCM:BURR-BROWN_SOT223, F.Cu at (182.1, 146.8)
- added J1: RJ45-HR911105A, USSTCM:HANRUN_RJ45, F.Cu at (159.8, 127.0)
- added J2: RJ45-HR911105A, USSTCM:HANRUN_RJ45, F.Cu at (159.8, 108.4)
- added JP1: Jumper_NC_Small, USST-footprints:J_0603, F.Cu at (251.2, 34.7)
- added P1: CONN_I2C, Pin_Headers:Pin_Header_Angled_1x04_Pitch2.54mm, F.Cu at (222.7, -37.9)
- added P2: SERVO_PWM0, Pin_Headers:Pin_Header_Angled_1x03_Pitch2.54mm, F.Cu at (235.3, -37.9)
- added P3: SERVO_PWM1, Pin_Headers:Pin_Header_Angled_1x03_Pitch2.54mm, F.Cu at (209.9, -21.4)
- added P4: CONN_UART0, Pin_Headers:Pin_Header_Angled_1x04_Pitch2.54mm, F.Cu at (222.7, -23.8)
- added P5: CONN_UART1_3DR, Pin_Headers:Pin_Header_Angled_1x06_Pitch2.54mm, F.Cu at (196.8, -37.9)
- added P6: CAN_CONN_01X04, Pin_Headers:Pin_Header_Angled_1x04_Pitch2.54mm, F.Cu at (256.8, 20.6)
- added P7: 5V POWER CONN, Connect:bornier2, F.Cu at (160.9, 146.7)
- added Q5: FDS6681Z, Housings_SOIC:SOIC-8_3.9x4.9mm_Pitch1.27mm, F.Cu at (160.9, 157.3)
- added R15: 49.9, Resistors_SMD:R_0805, F.Cu at (23.5, 162.3)
- added R16: 12k4, Resistors_SMD:R_0805, F.Cu at (31.4, 140.6)
- added R17: 12k, Resistors_SMD:R_0805, F.Cu at (42.9, 137.4)
- added R22: 1k8, Resistors_SMD:R_0805, F.Cu at (199.5, -19.3)
- added R23: 1k8, Resistors_SMD:R_0805, F.Cu at (196.1, -19.3)
- added R24: 100, Resistors_SMD:R_0805, F.Cu at (273.7, 20.0)
- added R36: 10k, Resistors_SMD:R_0805, F.Cu at (232.6, 9.23)
- added R38: 50, Resistors_SMD:R_0805, F.Cu at (239.5, 9.23)
- added R40: 50, Resistors_SMD:R_0805, F.Cu at (230.1, 14.6)
- added R41: 50, Resistors_SMD:R_0805, F.Cu at (233.6, 14.6)
- added R42: 1k, Resistors_SMD:R_0805, F.Cu at (225.8, 19.9)
- added R43: 1k, Resistors_SMD:R_0805, F.Cu at (225.7, 9.23)
- added SP1: SPEAKER, USST-footprints:AI-3035-TWT, F.Cu at (190.5, -66.7)
- added USB2: USB2, USST-footprints:USB-A-UPRIGHT, F.Cu at (89.8, 147.3)
- added USB3: USB2, USST-footprints:USB-A-UPRIGHT, F.Cu at (99.3, 147.3)
- added USB4: USB2, USST-footprints:USB-A-UPRIGHT, F.Cu at (108.5, 147.3)
- added USB5: USB2, USST-footprints:USB-A-UPRIGHT, F.Cu at (118.0, 147.3)
- C1, C41, C46: footprint USSTCM:RCL_C0805 -> Capacitors_SMD:C_0805
- C10, C11, C12, C17, C18, C19, C9: value 10u -> 100n; footprint USSTCM:RCL_C0805 -> Capacitors_SMD:C_0805
- C13, C14, C16, C25, C28, C29, C31, C32, C33, C38, C39, C4, C40: footprint USSTCM:RCL_C0603 -> Capacitors_SMD:C_0805
- C15, C23, C24: value 20p -> 100n; footprint USSTCM:RCL_C0603 -> Capacitors_SMD:C_0805
- C2: value 10u -> 20p; footprint USSTCM:RCL_C0805 -> Capacitors_SMD:C_0805
- C20: value 10u -> 1u; footprint USSTCM:RCL_C0805 -> Capacitors_SMD:C_0805
- C21, C22, C45: value 20p -> 10u; footprint USSTCM:RCL_C0603 -> Capacitors_SMD:C_0805
- C26, C27, C30, C34, C49: value 100n -> 10u; footprint USSTCM:RCL_C0603 -> Capacitors_SMD:C_0805
- C35, C36, C37: value 100n -> 0.1u; footprint USSTCM:RCL_C0603 -> Capacitors_SMD:C_0805
- C42: value 1u -> 10u; footprint USSTCM:RCL_C0805 -> Capacitors_SMD:C_0805
- C43: value 100n -> ~; footprint USSTCM:RCL_C0603 -> Capacitors_SMD:C_0805
- C44: value 20p -> ~; footprint USSTCM:RCL_C0603 -> Capacitors_SMD:C_0805
- C6, C8: value ~ -> 20p; footprint USSTCM:RCL_153CLV-0605 -> Capacitors_SMD:C_0805
- C7: value 100n -> 20p; footprint USSTCM:RCL_C0603 -> Capacitors_SMD:C_0805
- CAM1: value RASPI_CAM -> FFC-15; footprint USSTCM:RASPI_FFC-15 -> USST-footprints:FFC-15-PICAM
- FB1, FB2: footprint USSTCM:RASPI_C0805 -> Capacitors_SMD:C_0805
- IC1: value REG1117 -> FSUSB42MSOP10; footprint USSTCM:BURR-BROWN_SOT223 -> Housings_SSOP:MSOP-10_3x3mm_Pitch0.5mm
- IC2: value REG1117 -> RASPI_LAN9514; footprint USSTCM:BURR-BROWN_SOT223 -> Housings_DFN_QFN:QFN-64-1EP_9x9mm_Pitch0.5mm
- IC3: value RASPI_LAN9514 -> REG1117; footprint USSTCM:RASPI_QFN64-9X9 -> USSTCM:BURR-BROWN_SOT223
- IC5: value FSUSB42MSOP10 -> ENC28J60; footprint USSTCM:RASPI_MSOP10 -> Housings_SSOP:SSOP-28_5.3x10.2mm_Pitch0.65mm
- PWR1: footprint USSTCM:LED_CHIP-LED0603 -> Diodes_SMD:D_0805
- R1, R2: value 47k -> 100k; footprint USSTCM:RCL_R0603 -> Resistors_SMD:R_0805
- R10, R4, R5: value 100k -> 47k; footprint USSTCM:RCL_R0603 -> Resistors_SMD:R_0805
- R11: value 1k8 -> 10; footprint USSTCM:RCL_R0603 -> Resistors_SMD:R_0805
- R12, R14: value 1k8 -> 49.9; footprint USSTCM:RCL_R0603 -> Resistors_SMD:R_0805
- R13: value 1M -> 49.9; footprint USSTCM:RCL_R0603 -> Resistors_SMD:R_0805
- R18, R19: value 1k8 -> 12k; footprint USSTCM:RCL_R0603 -> Resistors_SMD:R_0805
- R20, R25, R3, R34, R6: footprint USSTCM:RCL_R0603 -> Resistors_SMD:R_0805
- R21: value 1k8 -> 400; footprint USSTCM:RCL_R0603 -> Resistors_SMD:R_0805
- R26: value 1k -> 100k; footprint USSTCM:RCL_R0603 -> Resistors_SMD:R_0805
- R27: value 10 -> 1k8; footprint USSTCM:RCL_R0603 -> Resistors_SMD:R_0805
- R28, R29, R30, R31: value 49.9 -> 1k8; footprint USSTCM:RCL_R0603 -> Resistors_SMD:R_0805
- R32: value 12k -> 1k8; footprint USSTCM:RCL_R0603 -> Resistors_SMD:R_0805
- R33: value 12k4 -> 100k; footprint USSTCM:RCL_R0603 -> Resistors_SMD:R_0805
- R35: value 1k8 -> 10k; footprint USSTCM:RCL_R0603 -> Resistors_SMD:R_0805
- R37: value 12k -> 50; footprint USSTCM:RCL_R0603 -> Resistors_SMD:R_0805
- R39: value 1k8 -> 2.32k; footprint USSTCM:RCL_R0603 -> Resistors_SMD:R_0805
- R7, R8: value 47k -> 1k; footprint USSTCM:RCL_R0603 -> Resistors_SMD:R_0805
- R9: value 12k -> 47k; footprint USSTCM:RCL_R0603 -> Resistors_SMD:R_0805
- U2: value MCP2515 -> MCP25625; footprint Housings_SOIC:SOIC-18_7.5x11.6mm_Pitch1.27mm -> Housings_SSOP:SSOP-28_5.3x10.2mm_Pitch0.65mm
- USB1: value MICRO_USB -> USB-TYPA; footprint USSTCM:MASTER_CLOCK_MICRO_USB -> USST-footprints:MINI-B-USBR
- moved R13 454.7 mm to (31.2, 146.0)
- moved C30 450.6 mm to (17.2, 163.0)
- moved C7 444.3 mm to (34.4, 161.7)
- moved FB1 443.2 mm to (6.22, 157.4)
- moved R20 441.2 mm to (6.03, 162.8)
- moved R11 440.9 mm to (31.2, 151.3)
- moved C11 440.5 mm to (38.7, 147.9)
- moved R8 436.8 mm to (42.2, 142.7)
- moved R9 432.7 mm to (46.3, 137.4)
- moved R7 430.2 mm to (54.8, 123.7)
- moved R12 426.3 mm to (34.9, 146.0)
- moved C31 421.0 mm to (13.2, 163.0)
- moved C4 414.3 mm to (50.1, 137.2)
- moved C22 408.5 mm to (46.4, 158.3)
- moved C12 405.2 mm to (50.3, 154.9)
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Connections:
- C1 pad 1: +5V -> +3V3
- C10 pad 1: 3V3 -> +3V3
- C11 pad 1: +5V -> GND
- C11 pad 2: GND -> Net-(C11-Pad2)
- C12 pad 1: +5V -> +3V3
- C13 pad 1: 3V3 -> GND
- C13 pad 2: GND -> (no net)
- C14 pad 1: /USSTCM LAN/5V_HDMI -> GND
- C14 pad 2: GND -> Net-(C11-Pad2)
- C15 pad 1: HDMI_CEC -> GND
- C15 pad 2: GND -> /USSTCM LAN/VDD18PLL
- C16 pad 2: 3V3 -> Net-(C11-Pad2)
- C17 pad 1: 1V8 -> GND
- C17 pad 2: GND -> Net-(C11-Pad2)
- C18 pad 1: 3V3 -> GND
- C18 pad 2: GND -> Net-(C11-Pad2)
- C19 pad 1: 1V8 -> GND
- C19 pad 2: GND -> Net-(C11-Pad2)
- C2 pad 1: +5V -> /HDMI_CEC
- C20 pad 1: 3V3 -> GND
- C20 pad 2: GND -> Net-(C20-Pad2)
- C21 pad 1: /USSTCM LAN/TX_P -> +5V
- C22 pad 1: /USSTCM LAN/TX_N -> +5V
- C23 pad 1: /USSTCM LAN/RX_P -> +3V3
- C24 pad 1: /USSTCM LAN/RX_N -> +3V3
- C25 pad 1: GND -> +3V3
- C25 pad 2: 3V3 -> GND
- C26 pad 1: /USSTCM LAN/N$17 -> +5V
- C27 pad 1: 3V3 -> +5V
- C28 pad 1: 3V3 -> GND
- C28 pad 2: GND -> /USSTCM LAN/VDD18CORE
- C29 pad 1: 3V3 -> GND
- C29 pad 2: GND -> /USSTCM LAN/VDD18CORE
- C30 pad 2: 3V3 -> /USSTCM LAN/VDD18CORE
- C31 pad 2: 3V3 -> +3V3
- C32 pad 2: /USSTCM LAN/3V3A -> +3V3
- C33 pad 2: /USSTCM LAN/3V3A -> +3V3
- C34 pad 2: /USSTCM LAN/3V3A -> +5V
- C35 pad 1: GND -> +3V3
- C35 pad 2: /USSTCM LAN/3V3A -> GND
- C36 pad 1: GND -> +5V
- C36 pad 2: /USSTCM LAN/3V3A -> GND
- C37 pad 1: GND -> +3V3
- C37 pad 2: /USSTCM LAN/3V3A -> GND
- C38 pad 2: /USSTCM LAN/3V3A -> +3V3
- C39 pad 2: /USSTCM LAN/VDD18CORE -> +3V3
- C4 pad 1: /USSTCM LAN/3V3A -> +3V3
- C40 pad 1: GND -> /USSTCM_VIDEO/5V_HDMI
- C40 pad 2: /USSTCM LAN/VDD18CORE -> GND
- C41 pad 1: GND -> +5V
- C41 pad 2: /USSTCM LAN/VDD18CORE -> GND
- C42 pad 1: GND -> +5V
- C42 pad 2: /USSTCM LAN/N$40 -> GND
- C43 pad 1: GND -> +1V8
- C43 pad 2: /USSTCM LAN/VDD18PLL -> GND
- C44 pad 1: GND -> +3V3
- C44 pad 2: /USSTCM LAN/XO -> GND
- C45 pad 1: GND -> +1V8
- C45 pad 2: /USSTCM LAN/XI -> GND
- C46 pad 1: 3V3 -> +3V3
- C49 pad 1: GND -> +3V3
- C49 pad 2: 3V3 -> GND
- C7 pad 1: /USSTCM LAN/3V3A -> /USSTCM LAN/ETH_RX_P
- C9 pad 1: 3V3 -> /USSTCM LAN/RCT
- D2 pad 2: /USSTCM LAN/5V_HDMI -> /USSTCM_VIDEO/5V_HDMI
- D2 pad 3: HDMI_SDA -> /HDMI_SCL
- D3 pad 2: /USSTCM LAN/5V_HDMI -> /USSTCM_VIDEO/5V_HDMI
- D3 pad 3: HDMI_SCL -> /HDMI_SDA
- D4 pad 2: /USSTCM LAN/5V_HDMI -> /USSTCM_VIDEO/5V_HDMI
- D4 pad 3: HDMI_CEC -> Net-(D4-Pad3)
- D5 pad 1: +5V -> /USSTCM_VIDEO/5V_HDMI
- D5 pad 2: (no net) -> +5V
- D5 pad 3: /USSTCM LAN/5V_HDMI -> (no net)
- FB1 pad 1: /USSTCM LAN/3V3A -> /USSTCM LAN/VDD18PLL
- FB1 pad 2: 3V3 -> Net-(C20-Pad2)
- FB2 pad 1: /USSTCM LAN/VDD18PLL -> Net-(C11-Pad2)
- FB2 pad 2: /USSTCM LAN/N$40 -> +3V3
- IC1 pad 1: GND -> +3V3
- IC1 pad 2: 1V8 -> Net-(IC1-Pad2)
- IC1 pad 3: +5V -> /USBD_P
- IC1 pad 4: (no net) -> /USBD_N
- IC2 pad 1: GND -> /USSTCM LAN/USB2_N
- IC2 pad 2: 3V3 -> /USSTCM LAN/USB2_P
- IC2 pad 3: +5V -> /USSTCM LAN/USB3_N
- IC2 pad 4: (no net) -> /USSTCM LAN/USB3_P
- IC3 pad 1: /USSTCM LAN/USBD2_N -> GND
- IC3 pad 2: /USSTCM LAN/USBD2_P -> +1V8
- IC3 pad 3: /USSTCM LAN/USBD3_N -> +5V
- IC3 pad 4: /USSTCM LAN/USBD3_P -> (no net)
- IC5 pad 1: 3V3 -> Net-(C50-Pad1)
- IC5 pad 10: GND -> Net-(IC5-Pad10)
- IC5 pad 2: /USSTCM LAN/N$29 -> GND
- IC5 pad 3: USBD_P -> (no net)
- IC5 pad 4: USBD_N -> /GPIO39
- IC5 pad 5: GND -> (no net)
- IC5 pad 6: /USSTCM LAN/USBDS_N -> /GPIO40
- IC5 pad 7: /USSTCM LAN/USBDS_P -> /GPIO41
- IC5 pad 8: /USSTCM LAN/USBDL_N -> /GPIO42
- IC5 pad 9: /USSTCM LAN/USBDL_P -> /GPIO45
- Q1 pad 1: VUSB_BOOT -> /VUSB_BOOT
- Q1 pad 2: /N$3 -> Net-(ACT1-Pad1)
- Q1 pad 3: /N$5 -> Net-(Q1-Pad3)
- Q2 pad 1: /N$6 -> Net-(Q2-Pad1)
- Q2 pad 2: /N$5 -> GND
- Q2 pad 3: GND -> Net-(ACT1-Pad1)
- Q3 pad 1: VUSB_BOOT -> /VUSB_BOOT
- Q3 pad 2: /USSTCM LAN/N$29 -> GND
- Q3 pad 3: GND -> Net-(IC1-Pad2)
- Q4 pad 1: /USSTCM LAN/N$34 -> Net-(D4-Pad3)
- Q4 pad 2: GPIO46 -> GND
- Q4 pad 3: GND -> /USSTCM_VIDEO/GPIO46
- R1 pad 2: VUSB_BOOT -> /GPIO29
- R10 pad 1: GPIO46 -> /VUSB_BOOT
- R10 pad 2: 1V8 -> GND
- R11 pad 1: HDMI_SDA -> /USSTCM LAN/RCT
- R11 pad 2: +5V -> +3V3
- R12 pad 1: HDMI_SCL -> +3V3
- R12 pad 2: +5V -> /USSTCM LAN/ETH_RX_N
- R13 pad 1: /USSTCM LAN/XO -> /USSTCM LAN/ETH_RX_P
- R13 pad 2: /USSTCM LAN/XI -> +3V3
- R14 pad 1: GPIO1 -> /USSTCM LAN/ETH_TX_N
- R14 pad 2: 3V3 -> +3V3
- R18 pad 1: 3V3 -> +3V3
- R18 pad 2: GPIO2 -> Net-(IC2-Pad41)
- R19 pad 1: 3V3 -> /GPIO6
- R19 pad 2: GPIO3 -> +3V3
- R2 pad 1: /N$6 -> GND
- R2 pad 2: 1V8 -> /GPIO44
- R20 pad 1: /USSTCM LAN/N$9 -> +3V3
- R20 pad 2: 3V3 -> Net-(IC2-Pad28)
- R21 pad 1: /N$1 -> Net-(R21-Pad1)
- R21 pad 2: 3V3 -> (no net)
- R25 pad 1: 3V3 -> Net-(R25-Pad1)
- R25 pad 2: /USSTCM LAN/N$7 -> GND
- R26 pad 1: 3V3 -> +3V3
- R26 pad 2: /USSTCM LAN/N$8 -> Net-(R26-Pad2)
- R27 pad 1: /USSTCM LAN/3V3A -> +3V3
- R27 pad 2: /USSTCM LAN/N$17 -> /GPIO28
- R28 pad 1: /USSTCM LAN/3V3A -> +3V3
- R28 pad 2: /USSTCM LAN/RX_N -> /GPIO0
- R29 pad 1: /USSTCM LAN/3V3A -> +3V3
- R29 pad 2: /USSTCM LAN/RX_P -> /GPIO29
- R3 pad 1: GPIO29 -> GND
- R3 pad 2: GND -> /GPIO28
- R30 pad 1: /USSTCM LAN/3V3A -> +3V3
- R30 pad 2: /USSTCM LAN/TX_N -> /GPIO1
- R31 pad 1: /USSTCM LAN/3V3A -> +5V
- R31 pad 2: /USSTCM LAN/TX_P -> /HDMI_SDA
- R32 pad 1: /USSTCM LAN/N$42 -> +5V
- R32 pad 2: 3V3 -> /HDMI_SCL
- R33 pad 1: /USSTCM LAN/N$43 -> +1V8
- R33 pad 2: GND -> /USSTCM_VIDEO/GPIO46
- R34 pad 1: GPIO0 -> +3V3
- R34 pad 2: 3V3 -> Net-(PWR1-Pad2)
- R35 pad 1: /N$4 -> +3V3
- R35 pad 2: 3V3 -> /GPIO45
- R37 pad 1: 3V3 -> /USSTCM_LAN2/RD+
- R37 pad 2: GPIO6 -> /USSTCM_LAN2/RCT
- R39 pad 1: GPIO28 -> Net-(IC5-Pad14)
- R39 pad 2: 3V3 -> GND
- R4 pad 1: GPIO28 -> /VUSB_BOOT
- R5 pad 1: /GPIO44 -> +1V8
- R5 pad 2: GND -> Net-(Q2-Pad1)
- R6 pad 1: GPIO29 -> +3V3
- R6 pad 2: 3V3 -> Net-(ACT1-Pad2)
- R7 pad 1: GND -> +3V3
- R7 pad 2: VUSB_BOOT -> Net-(J1-Pad12)
- R8 pad 1: /USSTCM LAN/N$29 -> +3V3
- R8 pad 2: 3V3 -> Net-(J1-Pad9)
- R9 pad 1: GND -> +3V3
- R9 pad 2: /USSTCM LAN/N$11 -> Net-(IC1-Pad2)
- U1 pad 11: GPIO3 -> (no net)
- U1 pad 111: HDMI_CK_N -> /HDMI_CK_N
- U1 pad 113: HDMI_CK_P -> /HDMI_CK_P
- U1 pad 117: HDMI_D0_N -> /HDMI_D0_N
- U1 pad 119: HDMI_D0_P -> /HDMI_D0_P
- U1 pad 123: HDMI_D1_N -> /HDMI_D1_N
- U1 pad 125: HDMI_D1_P -> /HDMI_D1_P
- U1 pad 129: HDMI_D2_N -> /HDMI_D2_N
- U1 pad 131: HDMI_D2_P -> /HDMI_D2_P
- U1 pad 136: CAM0_D0_P -> /CAM0_D0_P
- U1 pad 138: CAM0_D0_N -> /CAM0_D0_N
- U1 pad 142: CAM0_C_P -> /CAM0_C_P
- U1 pad 144: CAM0_C_N -> /CAM0_C_N
- U1 pad 147: CAM1_C_P -> /CAM1_C_P
- U1 pad 148: CAM0_D1_P -> /CAM0_D1_P
- U1 pad 149: CAM1_C_N -> /CAM1_C_N
- U1 pad 15: GPIO4 -> (no net)
- U1 pad 150: CAM0_D1_N -> /CAM0_D1_N
- U1 pad 153: CAM1_D1_P -> /CAM1_D1_P
- U1 pad 155: CAM1_D1_N -> /CAM1_D1_N
- U1 pad 159: CAM1_D0_P -> /CAM1_D0_P
- U1 pad 161: CAM1_D0_N -> /CAM1_D0_N
- U1 pad 165: USBD_P -> /USBD_P
- U1 pad 167: USBD_N -> /USBD_N
- U1 pad 17: GPIO5 -> /GPIO5
- U1 pad 171: HDMI_CEC -> /HDMI_CEC
- U1 pad 173: HDMI_SDA -> /HDMI_SDA
- U1 pad 175: HDMI_SCL -> /HDMI_SCL
- U1 pad 183: 1V8 -> +1V8
- U1 pad 184: 1V8 -> +1V8
- U1 pad 185: 1V8 -> +1V8
- U1 pad 186: 1V8 -> +1V8
- U1 pad 189: 3V3 -> +3V3
- U1 pad 190: 3V3 -> +3V3
- U1 pad 191: 3V3 -> +3V3
- U1 pad 192: 3V3 -> +3V3
- U1 pad 193: 3V3 -> +3V3
- U1 pad 194: 3V3 -> +3V3
- U1 pad 2: /N$3 -> Net-(Q1-Pad3)
- U1 pad 21: GPIO6 -> /GPIO6
- U1 pad 23: GPIO7 -> (no net)
- U1 pad 27: GPIO8 -> /GPIO8
- U1 pad 28: GPIO28 -> /GPIO28
- U1 pad 29: GPIO9 -> /GPIO9
- U1 pad 3: GPIO0 -> /GPIO0
- U1 pad 30: GPIO29 -> /GPIO29
- U1 pad 33: GPIO10 -> /GPIO10
- U1 pad 34: GPIO30 -> /GPIO30
- U1 pad 35: GPIO11 -> /GPIO11
- U1 pad 36: GPIO31 -> /GPIO31
- U1 pad 39: 3V3 -> +3V3
- U1 pad 40: 3V3 -> +3V3
- U1 pad 41: 3V3 -> +3V3
- U1 pad 42: 3V3 -> +3V3
- U1 pad 45: GPIO12 -> (no net)
- U1 pad 47: GPIO13 -> (no net)
- U1 pad 5: GPIO1 -> /GPIO1
- U1 pad 51: GPIO14 -> (no net)
- U1 pad 52: (no net) -> /GPIO34
- U1 pad 53: GPIO15 -> (no net)
- U1 pad 57: GPIO16 -> (no net)
- U1 pad 59: GPIO17 -> (no net)
- U1 pad 63: GPIO18 -> (no net)
- U1 pad 65: GPIO19 -> (no net)
- U1 pad 66: (no net) -> /GPIO39
- U1 pad 69: GPIO20 -> (no net)
- U1 pad 70: (no net) -> /GPIO40
- U1 pad 71: GPIO21 -> /GPIO21
- U1 pad 72: (no net) -> /GPIO41
- U1 pad 75: GPIO22 -> (no net)
- U1 pad 76: (no net) -> /GPIO42
- U1 pad 77: GPIO23 -> (no net)
- U1 pad 78: (no net) -> /GPIO43
- U1 pad 81: GPIO24 -> (no net)
- U1 pad 83: GPIO25 -> /GPIO25
- U1 pad 84: (no net) -> /GPIO45
- U1 pad 87: GPIO26 -> (no net)
- U1 pad 88: GPIO46 -> (no net)
- U1 pad 89: GPIO27 -> (no net)
- U1 pad 9: GPIO2 -> (no net)
- U1 pad 90: /N$6 -> Net-(Q2-Pad1)
- U2 pad 1: Net-(U2-Pad1) -> +3V3
- U2 pad 13: (no net) -> /GPIO25
- U2 pad 14: (no net) -> /GPIO11
- U2 pad 15: (no net) -> /GPIO10
- U2 pad 16: (no net) -> /GPIO9
- U2 pad 17: (no net) -> /GPIO8
- U2 pad 18: 3V3 -> Net-(R26-Pad2)
- U2 pad 2: Net-(U2-Pad2) -> (no net)
- U2 pad 3: (no net) -> /USSTCM_CAN_LITE/CAN_P
- U2 pad 4: (no net) -> /USSTCM_CAN_LITE/CAN_N
- U2 pad 5: (no net) -> Net-(R25-Pad1)
- U2 pad 9: GND -> /GPIO43
Routing:
- net /USSTCM LAN/USB_BOOT_N: track 0.00 -> 63.0 mm
- net /USSTCM LAN/USB_BOOT_P: track 0.00 -> 63.0 mm
- net /USSTCM LAN/USB2_N: track 0.00 -> 53.7 mm
- net /USSTCM LAN/USB2_P: track 0.00 -> 53.7 mm
- net /GPIO44: track 0.00 -> 50.2 mm, vias 0 -> 2
- net /USSTCM LAN/ETH_TX_P: track 0.00 -> 49.7 mm
- net /USSTCM LAN/ETH_TX_N: track 0.00 -> 49.7 mm
- net /USSTCM LAN/USB3_N: track 0.00 -> 44.1 mm
- net /USSTCM LAN/USB3_P: track 0.00 -> 44.1 mm
- net /USSTCM_LAN2/TD+: track 0.00 -> 39.2 mm
- net /USSTCM_LAN2/TD-: track 0.00 -> 39.2 mm
- net /GPIO40: track 0.00 -> 34.7 mm
- net /USSTCM LAN/USB4_N: track 0.00 -> 34.2 mm
- net /USSTCM LAN/USB4_P: track 0.00 -> 34.2 mm
- net /GPIO41: track 0.00 -> 33.8 mm
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Other:
- board outline removed
- net class Default: trace_width 0.25 -> 0.1524; via_dia 0.6 -> 0.6858; via_drill 0.4 -> 0.3302
