File: Projects/BatteryMount4/BatteryMount4.kicad_pcb (KiCad board)
At the start: 2 copper layers, 160 x 62 mm, 21 parts

Commit message: final edit on BatteryMount4
Parts:
- removed the REF** at (40.0, 3.62)
- removed the REF** at (117.4, 26.8)
- removed the REF** at (117.5, 19.1)
- removed the REF** at (117.5, 11.4)
- removed the REF** at (39.9, 57.8)
- removed the REF** at (39.9, 50.1)
- removed the REF** at (39.9, 42.3)
- removed the REF** at (39.9, 34.6)
- removed the REF** at (39.9, 26.8)
- removed the REF** at (40.0, 19.1)
- removed the REF** at (40.0, 11.4)
- removed the REF** at (117.4, 57.8)
- removed the REF** at (117.4, 34.6)
- removed the REF** at (117.4, 42.3)
- removed the REF** at (117.4, 50.1)
- added REF**: batt_wedge, USST-footprints:batt_wedge, F.Cu at (42.2, 19.0)
- added REF**: batt_wedge, USST-footprints:batt_wedge, F.Cu at (119.7, 50.0)
- added REF**: batt_wedge, USST-footprints:batt_wedge, F.Cu at (119.7, 42.2)
- added REF**: batt_wedge, USST-footprints:batt_wedge, F.Cu at (119.7, 34.6)
- added REF**: batt_wedge, USST-footprints:batt_wedge, F.Cu at (119.7, 26.7)
- added REF**: batt_wedge, USST-footprints:batt_wedge, F.Cu at (119.7, 19.0)
- added REF**: batt_wedge, USST-footprints:batt_wedge, F.Cu at (42.2, 11.3)
- added REF**: batt_wedge, USST-footprints:batt_wedge, F.Cu at (42.1, 57.7)
- added REF**: batt_wedge, USST-footprints:batt_wedge, F.Cu at (42.2, 50.0)
- added REF**: batt_wedge, USST-footprints:batt_wedge, F.Cu at (42.2, 42.2)
- added REF**: batt_wedge, USST-footprints:batt_wedge, F.Cu at (42.2, 34.6)
- added REF**: batt_wedge, USST-footprints:batt_wedge, F.Cu at (42.2, 26.7)
- added REF**: batt_wedge, USST-footprints:batt_wedge, F.Cu at (119.7, 11.3)
- added REF**: batt_wedge, USST-footprints:batt_wedge, F.Cu at (119.7, 3.56)
- added REF**: batt_wedge, USST-footprints:batt_wedge, F.Cu at (119.6, 57.7)
- moved REF** 75.3 mm to (42.2, 3.56)
- moved REF** 7.56 mm to (154.9, 5.17)
- moved REF** 7.44 mm to (5.11, 5.03)
- moved REF** 7.33 mm to (154.9, 56.9)
- moved REF** 7.33 mm to (4.85, 56.9)
Routing:
- net (no net): track 919.5 -> 1315.1 mm
