File: Projects/Front Connector Board/Front Connector Board.sch (KiCad schematic (older format))
At the start: 14 parts, among them J1 Conn_02x09_Odd_Even, J2 Conn_02x09_Odd_Even, J3 Conn_02x09_Odd_Even, J4 Conn_02x09_Odd_Even, P1 CONN_02X04, P10 CONN_02X04, P2 CONN_02X04, P3 CONN_02X04, P4 CONN_02X04, P5 CONN_02X04, P6 CONN_02X04, P7 CONN_02X04, P8 CONN_02X04, P9 CONN_02X04

Commit message: Furthered dev of the front & back panel designs
Parts:
- added J5, J6: Conn_02x08_Odd_Even, Pin_Headers:Pin_Header_Angled_2x08_Pitch2.54mm, symbol Conn_02x08_Odd_Even
Connections:
- new net: J5.1 (Pin_1), J6.1 (Pin_1)
- new net: J5.10 (Pin_10), J6.10 (Pin_10)
- new net: J5.11 (Pin_11), J6.11 (Pin_11)
- new net: J5.12 (Pin_12), J6.12 (Pin_12)
- new net: J5.13 (Pin_13), J6.13 (Pin_13)
- new net: J5.14 (Pin_14), J6.14 (Pin_14)
- new net: J5.15 (Pin_15), J6.15 (Pin_15)
- new net: J5.16 (Pin_16), J6.16 (Pin_16)
- new net: J5.2 (Pin_2), J6.2 (Pin_2)
- new net: J5.3 (Pin_3), J6.3 (Pin_3)
- new net: J5.4 (Pin_4), J6.4 (Pin_4)
- new net: J5.5 (Pin_5), J6.5 (Pin_5)
- new net: J5.6 (Pin_6), J6.6 (Pin_6)
- new net: J5.7 (Pin_7), J6.7 (Pin_7)
- new net: J5.8 (Pin_8), J6.8 (Pin_8)
- new net: J5.9 (Pin_9), J6.9 (Pin_9)
Changed lines of the file:
@@
 Wire Wire Line
 	3350 4825 3250 4825
+$Comp
+L Conn_02x08_Odd_Even J5
+U 1 1 5AD53005
+P 4050 5400
+F 0 "J5" H 4100 5800 50  0000 C CNN
+F 1 "Conn_02x08_Odd_Even" H 4100 4900 50  0000 C CNN
+F 2 "Pin_Headers:Pin_Header_Angled_2x08_Pitch2.54mm" H 4050 5400 50  0001 C CNN
+F 3 "" H 4050 5400 50  0001 C CNN
+	1    4050 5400
+	1    0    0    -1
+$EndComp
+$Comp
+L Conn_02x08_Odd_Even J6
+U 1 1 5AD53094
+P 4850 5400
+F 0 "J6" H 4900 5800 50  0000 C CNN
+F 1 "Conn_02x08_Odd_Even" H 4900 4900 50  0000 C CNN
+F 2 "Pin_Headers:Pin_Header_Angled_2x08_Pitch2.54mm" H 4850 5400 50  0001 C CNN
+F 3 "" H 4850 5400 50  0001 C CNN
+	1    4850 5400
+	-1   0    0    -1
+$EndComp
+Wire Wire Line
+	4350 5100 4550 5100
+Wire Wire Line
+	4350 5200 4550 5200
+Wire Wire Line
+	4350 5300 4550 5300
+Wire Wire Line
+	4350 5400 4550 5400
+Wire Wire Line
+	4350 5500 4550 5500
+Wire Wire Line
+	4350 5600 4550 5600
+Wire Wire Line
+	4350 5700 4550 5700
+Wire Wire Line
+	4350 5800 4550 5800
+Wire Wire Line
+	5050 5800 5050 5850
+Wire Wire Line
+	5050 5850 3850 5850
+Wire Wire Line
+	3850 5850 3850 5800
+Wire Wire Line
+	3850 5700 3800 5700
+Wire Wire Line
+	3800 5700 3800 5900
+Wire Wire Line
+	3800 5900 5100 5900
+Wire Wire Line
+	5100 5900 5100 5700
+Wire Wire Line
+	5100 5700 5050 5700
+Wire Wire Line
+	5050 5600 5150 5600
+Wire Wire Line
+	5150 5600 5150 5950
+Wire Wire Line
+	5150 5950 3750 5950
+Wire Wire Line
+	3750 5950 3750 5600
+Wire Wire Line
+	3750 5600 3850 5600
+Wire Wire Line
+	3850 5500 3700 5500
+Wire Wire Line
+	3700 5500 3700 6000
+Wire Wire Line
+	3700 6000 5200 6000
+Wire Wire Line
+	5200 6000 5200 5500
+Wire Wire Line
+	5200 5500 5050 5500
+Wire Wire Line
+	5050 5100 5050 5050
+Wire Wire Line
+	5050 5050 3850 5050
+Wire Wire Line
+	3850 5050 3850 5100
+Wire Wire Line
+	3850 5200 3800 5200
+Wire Wire Line
+	3800 5200 3800 5000
+Wire Wire Line
+	3800 5000 5100 5000
+Wire Wire Line
+	5100 5000 5100 5200
+Wire Wire Line
+	5100 5200 5050 5200
+Wire Wire Line
+	5050 5300 5150 5300
+Wire Wire Line
+	5150 5300 5150 4950
+Wire Wire Line
+	5150 4950 3750 4950
+Wire Wire Line
+	3750 4950 3750 5300
+Wire Wire Line
+	3750 5300 3850 5300
+Wire Wire Line
+	3850 5400 3700 5400
+Wire Wire Line
+	3700 5400 3700 4900
+Wire Wire Line
+	3700 4900 5200 4900
+Wire Wire Line
+	5200 4900 5200 5400
+Wire Wire Line
+	5200 5400 5050 5400
 $EndSCHEMATC
