File: Projects/Motor Controllers/newBLDC/Hardware/design/STM32F4 64LQFP.sch (KiCad schematic (older format))
At the start: 15 parts, among them P2 SWD, U1 STM32F40X_LQFP64, X2 8MHz 10ppm

Commit message: Created the schematic for the motor driver
Need to do more research into the microcontroller and if its possible to place arduino on it before implementing it into the schematic.
Parts:
- X2: symbol CRYSTAL_SMD -> CRYSTAL_SMD-RESCUE-BLDC_4
Changed lines of the file:
@@
 $Bitmap
 Pos 1750 6700
-Scale 1,000000
+Scale 1.000000
 Data
 89 50 4E 47 0D 0A 1A 0A 00 00 00 0D 49 48 44 52 00 00 02 6A 00 00 02 41 08 02 00 00 00 79 DB 0E
@@
 00 00 00 50 18 A4 4F 00 00 00 40 61 90 3E 01 00 00 00 85 41 FA 04 00 00 00 14 06 E9 13 00 00 00
 50 18 A4 4F 00 00 00 40 61 90 3E 01 00 00 00 85 41 FA 04 00 00 00 14 F6 FF 00 CF 05 3E 3D 48 21
-47 45 00 00 00 00 49 45 4E 44 AE 42 60 82 00
+47 45 00 00 00 00 49 45 4E 44 AE 42 60 82
 EndData
 $EndBitmap
 $Bitmap
 Pos 3100 1050
-Scale 1,000000
+Scale 1.000000
 Data
 89 50 4E 47 0D 0A 1A 0A 00 00 00 0D 49 48 44 52 00 00 03 D4 00 00 00 CC 08 02 00 00 00 1D DB 7C
@@
 9D 20 C6 37 81 40 20 10 08 04 02 81 D0 4E 10 E3 9B 40 20 10 08 04 02 81 40 68 27 88 F1 4D 20 10
 08 04 02 81 40 20 B4 13 C4 F8 26 10 08 04 02 81 40 20 10 DA 89 FF 07 6E 76 4C 5E B7 9B F3 6C 00
-00 00 00 49 45 4E 44 AE 42 60 82 05
+00 00 00 49 45 4E 44 AE 42 60 82
 EndData
 $EndBitmap
@@
 LED_GREEN
 $Comp
-L CRYSTAL_SMD X2
+L CRYSTAL_SMD-RESCUE-BLDC_4 X2
 U 1 1 540978A3
 P 7750 2050
