File: Projects/Arm/ArmPowerBoardV3/ArmPowerBoardV3/ArmPowerBoardV3.sch (KiCad schematic (older format))
At the start: 27 parts, among them J1 Screw_Terminal_01x04, J10 Atmega Holder, J11 Female Header R, J12 GPIO R, J13 JST serial, J2 Barrel_Jack, J3 Barrel_Jack, J4 Screw_Terminal_01x02, J5 Barrel_Jack, J6 Barrel_Jack, J7 Barrel_Jack, J8 Gpio L, J9 Femal header L, U1 ACS758, U2 VHB200W-Q24-S12, U3 25WDe-Swadj3, U4 Temp sense, Y1 Crystal

Commit message: work some more on the layout, had to move gpio for breakout board still need to hook those up and account for board mounting
Parts:
- removed BT1: 24V IN, TerminalBlocks:TerminalBlock_Big2pin, symbol Device:Battery
- removed J12: GPIO R, Connector_PinHeader_2.54mm:PinHeader_1x14_P2.54mm_Vertical, symbol Connector:Screw_Terminal_01x14
- removed J8: Gpio L, Connector_PinHeader_2.54mm:PinHeader_1x14_P2.54mm_Vertical, symbol Connector:Screw_Terminal_01x14
- removed R1: 15ohm, Resistor_SMD:R_0402_1005Metric, symbol Device:R
- removed U3: 25WDe-Swadj3, Converter_DCDC:Converter_DCDC_RECOM_R-78HBxx-0.5_THT, symbol De-Swadj~3:25WDe-Swadj3
- added BT1: 24vin, TerminalBlocks:TerminalBlock_1x02_P5.08mm_Horizontal, symbol Connector:Screw_Terminal_01x02
- added C10, C11, C7, C9: 100nF, Capacitor_SMD:C_0805_2012Metric_Pad1.15x1.40mm_HandSolder, symbol Device:C
- added C5, C6: 10pF, Capacitor_SMD:C_0805_2012Metric_Pad1.15x1.40mm_HandSolder, symbol Device:C
- added C8: 10 uF, Capacitor_SMD:C_0805_2012Metric_Pad1.15x1.40mm_HandSolder, symbol Device:C
- added J8: Gpio out, Connector_PinHeader_2.54mm:PinHeader_2x10_P2.54mm_Vertical, symbol Connector_Generic:Conn_02x10_Counter_Clockwise
- added U3: V7805-1000, TerminalBlocks:V7805-1000, symbol Regulator_Switching:R-78B5.0-2.0
- C2, C4: footprint Capacitor_THT:CP_Radial_Tantal_D4.5mm_P2.50mm -> Capacitor_SMD:C_0805_2012Metric_Pad1.15x1.40mm_HandSolder
- J11: value Female Header R -> Breakout R
- J2, J3: footprint PJ-002BH:CUI_PJ-002BH -> Connector_BarrelJack:BarrelJack_Wuerth_6941xx301002
- J5, J6, J7: footprint PJ-007:CUI_PJ-007 -> Connector_BarrelJack:BarrelJack_Wuerth_6941xx301002
- J9: value Femal header L -> Breakout L
Connections:
- net labels added: 5v+, ONoff
- net labels removed: 5vPS
- wire segments 78 -> 135
- no-connect marks 37 -> 21
Other:
- note added: "12v Power Supply\n"
- note added: "5v Power Supply\n"
- note added: "Headers for USB breakoutboard"
- note added: "JST UART Port"
- note added: "MCU\n"
- note added: "Power OUT\n"
- note added: "change to 0805\n"
- note removed: "Power OUT"
- note removed: "Power Supplies"
